Commit message: add inertial for arm

File: src/mobile_lift_arm/urdf/robot_arm.xacro (robot description, xacro)
@@ -4,5 +4,9 @@
     <!-- Đế arm -->
     <link name="arm_base_link">
-      <inertial><mass value="3"/><inertia ixx="0.03" iyy="0.03" izz="0.03" ixy="0" ixz="0" iyz="0"/></inertial>
+      <inertial>
+        <origin xyz="0 0 0.05" rpy="0 0 0"/>
+        <mass value="3.0"/>
+        <inertia ixx="0.03" ixy="0" ixz="0" iyy="0.03" iyz="0" izz="0.03"/>
+      </inertial>
       <visual>
         <origin xyz="0 0 0.05" rpy="0 0 0"/>
@@ -21,7 +25,18 @@
     <!-- Khớp 1: yaw -->
     <link name="arm_shoulder_yaw_link">
-      <inertial><mass value="2"/></inertial>
-      <visual><geometry><box size="0.08 0.08 0.15"/></geometry><material name="orange"/></visual>
-      <collision><geometry><box size="0.08 0.08 0.15"/></geometry></collision>
+      <inertial>
+        <origin xyz="0 0 0.075" rpy="0 0 0"/>
+        <mass value="2.0"/>
+        <inertia ixx="0.02" ixy="0" ixz="0" iyy="0.02" iyz="0" izz="0.02"/>
+      </inertial>
+      <visual>
+        <origin xyz="0 0 0.075" rpy="0 0 0"/>
+        <geometry><box size="0.08 0.08 0.15"/></geometry>
+        <material name="orange"/>
+      </visual>
+      <collision>
+        <origin xyz="0 0 0.075" rpy="0 0 0"/>
+        <geometry><box size="0.08 0.08 0.15"/></geometry>
+      </collision>
     </link>
     <joint name="arm_shoulder_yaw_joint" type="revolute">
@@ -35,7 +50,18 @@
     <!-- Khớp 2: pitch -->
     <link name="arm_shoulder_pitch_link">
-      <inertial><mass value="2"/></inertial>
-      <visual><geometry><box size="0.08 0.25 0.08"/></geometry><material name="orange"/></visual>
-      <collision><geometry><box size="0.08 0.25 0.08"/></geometry></collision>
+      <inertial>
+        <origin xyz="0 0 0.125" rpy="0 0 0"/>
+        <mass value="2.0"/>
+        <inertia ixx="0.02" ixy="0" ixz="0" iyy="0.02" iyz="0" izz="0.02"/>
+      </inertial>
+      <visual>
+        <origin xyz="0 0 0.125" rpy="0 0 0"/>
+        <geometry><box size="0.08 0.25 0.08"/></geometry>
+        <material name="orange"/>
+      </visual>
+      <collision>
+        <origin xyz="0 0 0.125" rpy="0 0 0"/>
+        <geometry><box size="0.08 0.25 0.08"/></geometry>
+      </collision>
     </link>
     <joint name="arm_shoulder_pitch_joint" type="revolute">
@@ -49,7 +75,18 @@
     <!-- Khớp 3: elbow -->
     <link name="arm_elbow_link">
-      <inertial><mass value="1.5"/></inertial>
-      <visual><geometry><box size="0.06 0.22 0.06"/></geometry><material name="orange"/></visual>
-      <collision><geometry><box size="0.06 0.22 0.06"/></geometry></collision>
+      <inertial>
+        <origin xyz="0 0 0.11" rpy="0 0 0"/>
+        <mass value="1.5"/>
+        <inertia ixx="0.015" ixy="0" ixz="0" iyy="0.015" iyz="0" izz="0.015"/>
+      </inertial>
+      <visual>
+        <origin xyz="0 0 0.11" rpy="0 0 0"/>
+        <geometry><box size="0.06 0.22 0.06"/></geometry>
+        <material name="orange"/>
+      </visual>
+      <collision>
+        <origin xyz="0 0 0.11" rpy="0 0 0"/>
+        <geometry><box size="0.06 0.22 0.06"/></geometry>
+      </collision>
     </link>
     <joint name="arm_elbow_joint" type="revolute">
@@ -61,9 +98,20 @@
       <dynamics damping="0.3"/>
     </joint>
-    <!-- EE -->
+    <!-- End-effector -->
     <link name="ee_link">
-      <inertial><mass value="0.5"/></inertial>
-      <visual><origin xyz="0 0 0.11"/><geometry><sphere radius="0.03"/></geometry><material name="orange"/></visual>
-      <collision><origin xyz="0 0 0.11"/><geometry><sphere radius="0.03"/></geometry></collision>
+      <inertial>
+        <origin xyz="0 0 0.11" rpy="0 0 0"/>
+        <mass value="0.5"/>
+        <inertia ixx="0.005" ixy="0" ixz="0" iyy="0.005" iyz="0" izz="0.005"/>
+      </inertial>
+      <visual>
+        <origin xyz="0 0 0.11" rpy="0 0 0"/>
+        <geometry><sphere radius="0.03"/></geometry>
+        <material name="orange"/>
+      </visual>
+      <collision>
+        <origin xyz="0 0 0.11" rpy="0 0 0"/>
+        <geometry><sphere radius="0.03"/></geometry>
+      </collision>
     </link>
     <joint name="ee_fixed" type="fixed">

Commit message: run ok v2

File: src/mobile_lift_arm/urdf/robot_arm.xacro (robot description, xacro)
@@ -2,11 +2,6 @@
 <robot xmlns:xacro="http://www.ros.org/wiki/xacro">
   <xacro:macro name="robot_arm" params="parent">
-    <!-- Đế arm -->
     <link name="arm_base_link">
-      <inertial>
-        <origin xyz="0 0 0.05" rpy="0 0 0"/>
-        <mass value="3.0"/>
-        <inertia ixx="0.03" ixy="0" ixz="0" iyy="0.03" iyz="0" izz="0.03"/>
-      </inertial>
+      <inertial><mass value="3"/><inertia ixx="0.03" iyy="0.03" izz="0.03" ixy="0" ixz="0" iyz="0"/></inertial>
       <visual>
         <origin xyz="0 0 0.05" rpy="0 0 0"/>
@@ -23,21 +18,5 @@
       <child link="arm_base_link"/>
     </joint>
-    <!-- Khớp 1: yaw -->
-    <link name="arm_shoulder_yaw_link">
-      <inertial>
-        <origin xyz="0 0 0.075" rpy="0 0 0"/>
-        <mass value="2.0"/>
-        <inertia ixx="0.02" ixy="0" ixz="0" iyy="0.02" iyz="0" izz="0.02"/>
-      </inertial>
-      <visual>
-        <origin xyz="0 0 0.075" rpy="0 0 0"/>
-        <geometry><box size="0.08 0.08 0.15"/></geometry>
-        <material name="orange"/>
-      </visual>
-      <collision>
-        <origin xyz="0 0 0.075" rpy="0 0 0"/>
-        <geometry><box size="0.08 0.08 0.15"/></geometry>
-      </collision>
-    </link>
+    <link name="arm_shoulder_yaw_link"/>
     <joint name="arm_shoulder_yaw_joint" type="revolute">
       <parent link="arm_base_link"/>
@@ -48,21 +27,5 @@
       <dynamics damping="0.3"/>
     </joint>
-    <!-- Khớp 2: pitch -->
-    <link name="arm_shoulder_pitch_link">
-      <inertial>
-        <origin xyz="0 0 0.125" rpy="0 0 0"/>
-        <mass value="2.0"/>
-        <inertia ixx="0.02" ixy="0" ixz="0" iyy="0.02" iyz="0" izz="0.02"/>
-      </inertial>
-      <visual>
-        <origin xyz="0 0 0.125" rpy="0 0 0"/>
-        <geometry><box size="0.08 0.25 0.08"/></geometry>
-        <material name="orange"/>
-      </visual>
-      <collision>
-        <origin xyz="0 0 0.125" rpy="0 0 0"/>
-        <geometry><box size="0.08 0.25 0.08"/></geometry>
-      </collision>
-    </link>
+    <link name="arm_shoulder_pitch_link"/>
     <joint name="arm_shoulder_pitch_joint" type="revolute">
       <parent link="arm_shoulder_yaw_link"/>
@@ -73,21 +36,5 @@
       <dynamics damping="0.3"/>
     </joint>
-    <!-- Khớp 3: elbow -->
-    <link name="arm_elbow_link">
-      <inertial>
-        <origin xyz="0 0 0.11" rpy="0 0 0"/>
-        <mass value="1.5"/>
-        <inertia ixx="0.015" ixy="0" ixz="0" iyy="0.015" iyz="0" izz="0.015"/>
-      </inertial>
-      <visual>
-        <origin xyz="0 0 0.11" rpy="0 0 0"/>
-        <geometry><box size="0.06 0.22 0.06"/></geometry>
-        <material name="orange"/>
-      </visual>
-      <collision>
-        <origin xyz="0 0 0.11" rpy="0 0 0"/>
-        <geometry><box size="0.06 0.22 0.06"/></geometry>
-      </collision>
-    </link>
+    <link name="arm_elbow_link"/>
     <joint name="arm_elbow_joint" type="revolute">
       <parent link="arm_shoulder_pitch_link"/>
@@ -98,21 +45,5 @@
       <dynamics damping="0.3"/>
     </joint>
-    <!-- End-effector -->
-    <link name="ee_link">
-      <inertial>
-        <origin xyz="0 0 0.11" rpy="0 0 0"/>
-        <mass value="0.5"/>
-        <inertia ixx="0.005" ixy="0" ixz="0" iyy="0.005" iyz="0" izz="0.005"/>
-      </inertial>
-      <visual>
-        <origin xyz="0 0 0.11" rpy="0 0 0"/>
-        <geometry><sphere radius="0.03"/></geometry>
-        <material name="orange"/>
-      </visual>
-      <collision>
-        <origin xyz="0 0 0.11" rpy="0 0 0"/>
-        <geometry><sphere radius="0.03"/></geometry>
-      </collision>
-    </link>
+    <link name="ee_link"/>
     <joint name="ee_fixed" type="fixed">
       <parent link="arm_elbow_link"/>

Commit message: Fix: Correct parent parameter syntax in arm_base_mount joint

File: src/mobile_lift_arm/urdf/robot_arm.xacro (robot description, xacro)
@@ -293,7 +293,7 @@
     </visual>
 </link>
-    <!-- Mount to parent (e.g., lift_top_link) -->
+    <!-- Mount the arm on the given parent -->
     <joint name="arm_base_mount" type="fixed">
-      <parent link="{parent}"/>
+      <parent link="${parent}"/>
       <child link="arm_base_link"/>
       <origin xyz="0 0 0" rpy="0 0 0"/>

Commit message: Fix: Update arm joint names to match control commands

File: src/mobile_lift_arm/urdf/robot_arm.xacro (robot description, xacro)
@@ -39,5 +39,5 @@
     </visual>
 </link>
-<joint name="arm_j1" type="revolute">
+<joint name="arm_shoulder_yaw_joint" type="revolute">
     <origin xyz="0.0 0.0 0.0" rpy="0.0 0.0 0.0"/>
     <parent link="arm_l0"/>
@@ -102,5 +102,5 @@
     </visual>
 </link>
-<joint name="arm_j2" type="revolute">
+<joint name="arm_shoulder_pitch_joint" type="revolute">
     <origin xyz="0.25 0.0 0.0" rpy="0.0 ${pi/2} 0.0"/>
     <parent link="arm_l2"/>
@@ -134,5 +134,5 @@
     </visual>
 </link>
-<joint name="arm_j3" type="revolute">
+<joint name="arm_shoulder_roll_joint" type="revolute">
     <origin xyz="-0.30 0.0 0.0" rpy="0.0 0.0 0.0"/>
     <parent link="arm_l3"/>
@@ -197,5 +197,5 @@
     </visual>
 </link>
-<joint name="arm_j4" type="revolute">
+<joint name="arm_elbow_pitch_joint" type="revolute">
     <origin xyz="-0.32 0.0 0.0" rpy="0.0 0.0 0.0"/>
     <parent link="arm_l5"/>
@@ -229,5 +229,5 @@
     </visual>
 </link>
-<joint name="arm_j5" type="revolute">
+<joint name="arm_wrist_pitch_joint" type="revolute">
     <origin xyz="0.0 0.0 0.25" rpy="0.0 ${-pi/2} ${2*pi}"/>
     <parent link="arm_l6"/>
@@ -261,5 +261,5 @@
     </visual>
 </link>
-<joint name="arm_j6" type="revolute">
+<joint name="arm_wrist_roll_joint" type="revolute">
     <origin xyz="0.0 0.0 0.18" rpy="0.0 ${pi/2} 0.0"/>
     <parent link="arm_le"/>
