Commit message: launch ok - v1 - show on gazebo

File: src/mobile_lift_arm/urdf/base_vehicle.xacro (robot description, xacro)
@@ -1,37 +1,41 @@
 <?xml version="1.0"?>
 <robot xmlns:xacro="http://www.ros.org/wiki/xacro">
-  <xacro:macro name="base_vehicle" params="prefix:= base_width:=0.6 base_length:=0.8 base_height:=0.15 wheel_radius:=0.1 wheel_thickness:=0.05">
-    <!-- Base link -->
-    <link name="${prefix}base_link">
+  <!-- Properties cố định để tránh lỗi tham số -->
+  <xacro:property name="BASE_LENGTH" value="0.8"/>
+  <xacro:property name="BASE_WIDTH"  value="0.6"/>
+  <xacro:property name="BASE_HEIGHT" value="0.15"/>
+  <xacro:property name="WHEEL_RADIUS" value="0.1"/>
+  <xacro:property name="WHEEL_THICK"  value="0.05"/>
+  <xacro:macro name="base_vehicle" params="">
+    <link name="base_link">
       <inertial>
-        <origin xyz="0 0 ${base_height/2}" rpy="0 0 0"/>
+        <origin xyz="0 0 ${BASE_HEIGHT/2}" rpy="0 0 0"/>
         <mass value="20.0"/>
         <inertia ixx="0.6" ixy="0" ixz="0" iyy="0.6" iyz="0" izz="0.6"/>
       </inertial>
       <visual>
-        <origin xyz="0 0 ${base_height/2}" rpy="0 0 0"/>
+        <origin xyz="0 0 ${BASE_HEIGHT/2}" rpy="0 0 0"/>
         <geometry>
-          <box size="${base_length} ${base_width} ${base_height}"/>
+          <box size="${BASE_LENGTH} ${BASE_WIDTH} ${BASE_HEIGHT}"/>
         </geometry>
         <material name="gray"><color rgba="0.5 0.5 0.5 1"/></material>
       </visual>
       <collision>
-        <origin xyz="0 0 ${base_height/2}" rpy="0 0 0"/>
+        <origin xyz="0 0 ${BASE_HEIGHT/2}" rpy="0 0 0"/>
         <geometry>
-          <box size="${base_length} ${base_width} ${base_height}"/>
+          <box size="${BASE_LENGTH} ${BASE_WIDTH} ${BASE_HEIGHT}"/>
         </geometry>
       </collision>
     </link>
-    <!-- Wheels (left/right) -->
     <link name="left_wheel_link">
       <inertial><mass value="2"/><inertia ixx="0.02" iyy="0.02" izz="0.02" ixy="0" ixz="0" iyz="0"/></inertial>
       <visual>
-        <origin xyz="0 ${base_width/2 + wheel_thickness/2} ${wheel_radius}" rpy="0 1.5708 0"/>
-        <geometry><cylinder radius="${wheel_radius}" length="${wheel_thickness}"/></geometry>
+        <origin xyz="0 ${BASE_WIDTH/2 + WHEEL_THICK/2} ${WHEEL_RADIUS}" rpy="0 1.5708 0"/>
+        <geometry><cylinder radius="${WHEEL_RADIUS}" length="${WHEEL_THICK}"/></geometry>
         <material name="black"><color rgba="0.1 0.1 0.1 1"/></material>
       </visual>
       <collision>
-        <origin xyz="0 ${base_width/2 + wheel_thickness/2} ${wheel_radius}" rpy="0 1.5708 0"/>
-        <geometry><cylinder radius="${wheel_radius}" length="${wheel_thickness}"/></geometry>
+        <origin xyz="0 ${BASE_WIDTH/2 + WHEEL_THICK/2} ${WHEEL_RADIUS}" rpy="0 1.5708 0"/>
+        <geometry><cylinder radius="${WHEEL_RADIUS}" length="${WHEEL_THICK}"/></geometry>
       </collision>
     </link>
@@ -39,24 +43,24 @@
       <inertial><mass value="2"/><inertia ixx="0.02" iyy="0.02" izz="0.02" ixy="0" ixz="0" iyz="0"/></inertial>
       <visual>
-        <origin xyz="0 -${base_width/2 + wheel_thickness/2} ${wheel_radius}" rpy="0 1.5708 0"/>
-        <geometry><cylinder radius="${wheel_radius}" length="${wheel_thickness}"/></geometry>
+        <origin xyz="0 -${BASE_WIDTH/2 + WHEEL_THICK/2} ${WHEEL_RADIUS}" rpy="0 1.5708 0"/>
+        <geometry><cylinder radius="${WHEEL_RADIUS}" length="${WHEEL_THICK}"/></geometry>
         <material name="black"><color rgba="0.1 0.1 0.1 1"/></material>
       </visual>
       <collision>
-        <origin xyz="0 -${base_width/2 + wheel_thickness/2} ${wheel_radius}" rpy="0 1.5708 0"/>
-        <geometry><cylinder radius="${wheel_radius}" length="${wheel_thickness}"/></geometry>
+        <origin xyz="0 -${BASE_WIDTH/2 + WHEEL_THICK/2} ${WHEEL_RADIUS}" rpy="0 1.5708 0"/>
+        <geometry><cylinder radius="${WHEEL_RADIUS}" length="${WHEEL_THICK}"/></geometry>
       </collision>
     </link>
     <joint name="left_wheel_joint" type="continuous">
-      <parent link="${prefix}base_link"/>
+      <parent link="base_link"/>
       <child link="left_wheel_link"/>
-      <origin xyz="0 ${base_width/2} ${wheel_radius}" rpy="0 0 0"/>
+      <origin xyz="0 ${BASE_WIDTH/2} ${WHEEL_RADIUS}" rpy="0 0 0"/>
       <axis xyz="0 1 0"/>
       <limit effort="10" velocity="20"/>
     </joint>
     <joint name="right_wheel_joint" type="continuous">
-      <parent link="${prefix}base_link"/>
+      <parent link="base_link"/>
       <child link="right_wheel_link"/>
-      <origin xyz="0 -${base_width/2} ${wheel_radius}" rpy="0 0 0"/>
+      <origin xyz="0 -${BASE_WIDTH/2} ${WHEEL_RADIUS}" rpy="0 0 0"/>
       <axis xyz="0 1 0"/>
       <limit effort="10" velocity="20"/>

File: src/mobile_lift_arm/urdf/mobile_lift_arm.urdf.xacro (robot description, xacro)
@@ -1,15 +1,14 @@
 <?xml version="1.0"?>
 <robot name="mobile_lift_arm" xmlns:xacro="http://www.ros.org/wiki/xacro">
-  <!-- Include modules -->
   <xacro:include filename="$(find mobile_lift_arm)/urdf/base_vehicle.xacro"/>
   <xacro:include filename="$(find mobile_lift_arm)/urdf/scissor_lift.xacro"/>
   <xacro:include filename="$(find mobile_lift_arm)/urdf/robot_arm.xacro"/>
   <!-- Base -->
-  <xacro:base_vehicle prefix=""/>
-  <!-- Lift mounted on base_link -->
+  <xacro:base_vehicle/>
+  <!-- Lift gắn trên base_link -->
   <xacro:scissor_lift parent="base_link"/>
-  <!-- 3-DOF Arm mounted on lift top -->
+  <!-- Arm gắn trên lift_top_link -->
   <xacro:robot_arm parent="lift_top_link"/>
-  <!-- Gazebo-ros2-control plugin -->
+  <!-- Gazebo ros2_control -->
   <gazebo>
     <plugin name="gazebo_ros2_control" filename="libgazebo_ros2_control.so">
@@ -17,10 +16,7 @@
     </plugin>
   </gazebo>
-  <!-- ros2_control interface -->
+  <!-- ros2_control -->
   <ros2_control name="GazeboSystem" type="system">
-    <hardware>
-      <plugin>gazebo_ros2_control/GazeboSystem</plugin>
-    </hardware>
-    <!-- diff drive joints (velocity cmd) -->
+    <hardware><plugin>gazebo_ros2_control/GazeboSystem</plugin></hardware>
     <joint name="left_wheel_joint">
       <command_interface name="velocity"/>
@@ -33,5 +29,4 @@
       <state_interface name="velocity"/>
     </joint>
-    <!-- lift prismatic (position cmd) -->
     <joint name="lift_joint">
       <command_interface name="position"/>
@@ -39,5 +34,4 @@
       <state_interface name="velocity"/>
     </joint>
-    <!-- arm (position cmd via trajectory controller) -->
     <joint name="arm_shoulder_yaw_joint">
       <command_interface name="position"/>
@@ -56,8 +50,3 @@
     </joint>
   </ros2_control>
-  <!-- Gazebo material friction etc. -->
-  <gazebo reference="base_link">
-    <kp>500000.0</kp>
-    <kd>10.0</kd>
-  </gazebo>
 </robot>

File: src/mobile_lift_arm/urdf/robot_arm.xacro (robot description, xacro)
@@ -14,12 +14,5 @@
       <child link="arm_base_link"/>
     </joint>
-    <!-- Joint 1: shoulder yaw -->
-    <link name="arm_shoulder_yaw_link">
-      <inertial><mass value="2"/><inertia ixx="0.02" iyy="0.02" izz="0.02" ixy="0" ixz="0" iyz="0"/></inertial>
-      <visual>
-        <geometry><box size="0.08 0.08 0.15"/></geometry>
-        <material name="orange"/>
-      </visual>
-    </link>
+    <link name="arm_shoulder_yaw_link"/>
     <joint name="arm_shoulder_yaw_joint" type="revolute">
       <parent link="arm_base_link"/>
@@ -30,12 +23,5 @@
       <dynamics damping="0.3"/>
     </joint>
-    <!-- Joint 2: shoulder pitch -->
-    <link name="arm_shoulder_pitch_link">
-      <inertial><mass value="2"/><inertia ixx="0.02" iyy="0.02" izz="0.02" ixy="0" ixz="0" iyz="0"/></inertial>
-      <visual>
-        <geometry><box size="0.08 0.25 0.08"/></geometry>
-        <material name="orange"/>
-      </visual>
-    </link>
+    <link name="arm_shoulder_pitch_link"/>
     <joint name="arm_shoulder_pitch_joint" type="revolute">
       <parent link="arm_shoulder_yaw_link"/>
@@ -46,12 +32,5 @@
       <dynamics damping="0.3"/>
     </joint>
-    <!-- Joint 3: elbow -->
-    <link name="arm_elbow_link">
-      <inertial><mass value="1.5"/><inertia ixx="0.015" iyy="0.015" izz="0.015" ixy="0" ixz="0" iyz="0"/></inertial>
-      <visual>
-        <geometry><box size="0.06 0.22 0.06"/></geometry>
-        <material name="orange"/>
-      </visual>
-    </link>
+    <link name="arm_elbow_link"/>
     <joint name="arm_elbow_joint" type="revolute">
       <parent link="arm_shoulder_pitch_link"/>
@@ -62,13 +41,5 @@
       <dynamics damping="0.3"/>
     </joint>
-    <!-- Simple end-effector -->
-    <link name="ee_link">
-      <inertial><mass value="0.5"/><inertia ixx="0.005" iyy="0.005" izz="0.005" ixy="0" ixz="0" iyz="0"/></inertial>
-      <visual>
-        <origin xyz="0 0 0.12" rpy="0 0 0"/>
-        <geometry><sphere radius="0.03"/></geometry>
-        <material name="orange"/>
-      </visual>
-    </link>
+    <link name="ee_link"/>
     <joint name="ee_fixed" type="fixed">
       <parent link="arm_elbow_link"/>

File: src/mobile_lift_arm/urdf/scissor_lift.xacro (robot description, xacro)
@@ -1,27 +1,25 @@
 <?xml version="1.0"?>
 <robot xmlns:xacro="http://www.ros.org/wiki/xacro">
-  <xacro:macro name="scissor_lift" params="parent lift_height_min:=0.0 lift_height_max:=1.2 top_size_xy:=0.5 top_thickness:=0.05">
-    <!-- Moving table (top platform) -->
+  <xacro:property name="LIFT_MIN" value="0.0"/>
+  <xacro:property name="LIFT_MAX" value="1.2"/>
+  <xacro:property name="TOP_XY"   value="0.5"/>
+  <xacro:property name="TOP_T"    value="0.05"/>
+  <xacro:macro name="scissor_lift" params="parent">
     <link name="lift_link">
       <inertial>
-        <origin xyz="0 0 ${top_thickness/2}" rpy="0 0 0"/>
+        <origin xyz="0 0 ${TOP_T/2}" rpy="0 0 0"/>
         <mass value="8.0"/>
         <inertia ixx="0.08" ixy="0" ixz="0" iyy="0.08" iyz="0" izz="0.08"/>
       </inertial>
       <visual>
-        <origin xyz="0 0 ${top_thickness/2}" rpy="0 0 0"/>
-        <geometry>
-          <box size="${top_size_xy} ${top_size_xy} ${top_thickness}"/>
-        </geometry>
+        <origin xyz="0 0 ${TOP_T/2}" rpy="0 0 0"/>
+        <geometry><box size="${TOP_XY} ${TOP_XY} ${TOP_T}"/></geometry>
         <material name="blue"><color rgba="0.2 0.3 0.9 1"/></material>
       </visual>
       <collision>
-        <origin xyz="0 0 ${top_thickness/2}" rpy="0 0 0"/>
-        <geometry>
-          <box size="${top_size_xy} ${top_size_xy} ${top_thickness}"/>
-        </geometry>
+        <origin xyz="0 0 ${TOP_T/2}" rpy="0 0 0"/>
+        <geometry><box size="${TOP_XY} ${TOP_XY} ${TOP_T}"/></geometry>
       </collision>
     </link>
-    <!-- Prismatic joint to simulate lift -->
     <joint name="lift_joint" type="prismatic">
       <parent link="${parent}"/>
@@ -29,15 +27,8 @@
       <origin xyz="0 0 0.15" rpy="0 0 0"/>
       <axis xyz="0 0 1"/>
-      <limit lower="${lift_height_min}" upper="${lift_height_max}" effort="500" velocity="0.2"/>
+      <limit lower="${LIFT_MIN}" upper="${LIFT_MAX}" effort="500" velocity="0.2"/>
       <dynamics damping="5.0" friction="0.1"/>
     </joint>
-    <!-- Top link for mounting the arm -->
-    <link name="lift_top_link">
-      <visual>
-        <origin xyz="0 0 ${top_thickness}" rpy="0 0 0"/>
-        <geometry><sphere radius="0.01"/></geometry>
-        <material name="invisible"><color rgba="0 0 0 0"/></material>
-      </visual>
-    </link>
+    <link name="lift_top_link"/>
     <joint name="lift_top_fixed" type="fixed">
       <parent link="lift_link"/>

Commit message: update

File: src/mobile_lift_arm/urdf/base_vehicle.xacro (robot description, xacro)
@@ -1,5 +1,5 @@
 <?xml version="1.0"?>
 <robot xmlns:xacro="http://www.ros.org/wiki/xacro">
-  <!-- Properties cố định để tránh lỗi tham số -->
+  <!-- Kích thước chuẩn -->
   <xacro:property name="BASE_LENGTH" value="0.8"/>
   <xacro:property name="BASE_WIDTH"  value="0.6"/>
@@ -8,4 +8,5 @@
   <xacro:property name="WHEEL_THICK"  value="0.05"/>
   <xacro:macro name="base_vehicle" params="">
+    <!-- Thân xe -->
     <link name="base_link">
       <inertial>
@@ -16,40 +17,39 @@
       <visual>
         <origin xyz="0 0 ${BASE_HEIGHT/2}" rpy="0 0 0"/>
-        <geometry>
-          <box size="${BASE_LENGTH} ${BASE_WIDTH} ${BASE_HEIGHT}"/>
-        </geometry>
+        <geometry><box size="${BASE_LENGTH} ${BASE_WIDTH} ${BASE_HEIGHT}"/></geometry>
         <material name="gray"><color rgba="0.5 0.5 0.5 1"/></material>
       </visual>
       <collision>
         <origin xyz="0 0 ${BASE_HEIGHT/2}" rpy="0 0 0"/>
-        <geometry>
-          <box size="${BASE_LENGTH} ${BASE_WIDTH} ${BASE_HEIGHT}"/>
-        </geometry>
+        <geometry><box size="${BASE_LENGTH} ${BASE_WIDTH} ${BASE_HEIGHT}"/></geometry>
       </collision>
     </link>
+    <!-- Bánh trái: frame bánh = child frame của joint, đặt visual/collision ở (0,0,0) -->
     <link name="left_wheel_link">
       <inertial><mass value="2"/><inertia ixx="0.02" iyy="0.02" izz="0.02" ixy="0" ixz="0" iyz="0"/></inertial>
       <visual>
-        <origin xyz="0 ${BASE_WIDTH/2 + WHEEL_THICK/2} ${WHEEL_RADIUS}" rpy="0 1.5708 0"/>
+        <origin xyz="0 0 0" rpy="0 1.5708 0"/>
         <geometry><cylinder radius="${WHEEL_RADIUS}" length="${WHEEL_THICK}"/></geometry>
         <material name="black"><color rgba="0.1 0.1 0.1 1"/></material>
       </visual>
       <collision>
-        <origin xyz="0 ${BASE_WIDTH/2 + WHEEL_THICK/2} ${WHEEL_RADIUS}" rpy="0 1.5708 0"/>
+        <origin xyz="0 0 0" rpy="0 1.5708 0"/>
         <geometry><cylinder radius="${WHEEL_RADIUS}" length="${WHEEL_THICK}"/></geometry>
       </collision>
     </link>
+    <!-- Bánh phải -->
     <link name="right_wheel_link">
       <inertial><mass value="2"/><inertia ixx="0.02" iyy="0.02" izz="0.02" ixy="0" ixz="0" iyz="0"/></inertial>
       <visual>
-        <origin xyz="0 -${BASE_WIDTH/2 + WHEEL_THICK/2} ${WHEEL_RADIUS}" rpy="0 1.5708 0"/>
+        <origin xyz="0 0 0" rpy="0 1.5708 0"/>
         <geometry><cylinder radius="${WHEEL_RADIUS}" length="${WHEEL_THICK}"/></geometry>
         <material name="black"><color rgba="0.1 0.1 0.1 1"/></material>
       </visual>
       <collision>
-        <origin xyz="0 -${BASE_WIDTH/2 + WHEEL_THICK/2} ${WHEEL_RADIUS}" rpy="0 1.5708 0"/>
+        <origin xyz="0 0 0" rpy="0 1.5708 0"/>
         <geometry><cylinder radius="${WHEEL_RADIUS}" length="${WHEEL_THICK}"/></geometry>
       </collision>
     </link>
+    <!-- Joint đặt vị trí bánh: ±y và z = bán kính -->
     <joint name="left_wheel_joint" type="continuous">
       <parent link="base_link"/>
@@ -66,4 +66,14 @@
       <limit effort="10" velocity="20"/>
     </joint>
+    <!-- Ma sát để bánh bám sàn -->
+    <gazebo reference="left_wheel_link">
+      <mu1>1.2</mu1><mu2>1.2</mu2>
+    </gazebo>
+    <gazebo reference="right_wheel_link">
+      <mu1>1.2</mu1><mu2>1.2</mu2>
+    </gazebo>
+    <gazebo reference="base_link">
+      <mu1>0.8</mu1><mu2>0.8</mu2>
+    </gazebo>
   </xacro:macro>
 </robot>

File: src/mobile_lift_arm/urdf/mobile_lift_arm.urdf.xacro (robot description, xacro)
@@ -13,4 +13,6 @@
   <gazebo>
     <plugin name="gazebo_ros2_control" filename="libgazebo_ros2_control.so">
+      <!-- ép namespace khớp với -entity -->
+      <robotNamespace>/mobile_lift_arm</robotNamespace>
       <parameters>$(find mobile_lift_arm)/config/ros2_controllers.yaml</parameters>
     </plugin>

File: src/mobile_lift_arm/urdf/robot_arm.xacro (robot description, xacro)
@@ -2,4 +2,5 @@
 <robot xmlns:xacro="http://www.ros.org/wiki/xacro">
   <xacro:macro name="robot_arm" params="parent">
+    <!-- Đế arm -->
     <link name="arm_base_link">
       <inertial><mass value="3"/><inertia ixx="0.03" iyy="0.03" izz="0.03" ixy="0" ixz="0" iyz="0"/></inertial>
@@ -9,4 +10,8 @@
         <material name="orange"><color rgba="0.9 0.5 0.2 1"/></material>
       </visual>
+      <collision>
+        <origin xyz="0 0 0.05" rpy="0 0 0"/>
+        <geometry><cylinder radius="0.06" length="0.1"/></geometry>
+      </collision>
     </link>
     <joint name="arm_base_fixed" type="fixed">
@@ -14,5 +19,10 @@
       <child link="arm_base_link"/>
     </joint>
-    <link name="arm_shoulder_yaw_link"/>
+    <!-- Khớp 1: yaw -->
+    <link name="arm_shoulder_yaw_link">
+      <inertial><mass value="2"/></inertial>
+      <visual><geometry><box size="0.08 0.08 0.15"/></geometry><material name="orange"/></visual>
+      <collision><geometry><box size="0.08 0.08 0.15"/></geometry></collision>
+    </link>
     <joint name="arm_shoulder_yaw_joint" type="revolute">
       <parent link="arm_base_link"/>
@@ -23,5 +33,10 @@
       <dynamics damping="0.3"/>
     </joint>
-    <link name="arm_shoulder_pitch_link"/>
+    <!-- Khớp 2: pitch -->
+    <link name="arm_shoulder_pitch_link">
+      <inertial><mass value="2"/></inertial>
+      <visual><geometry><box size="0.08 0.25 0.08"/></geometry><material name="orange"/></visual>
+      <collision><geometry><box size="0.08 0.25 0.08"/></geometry></collision>
+    </link>
     <joint name="arm_shoulder_pitch_joint" type="revolute">
       <parent link="arm_shoulder_yaw_link"/>
@@ -32,5 +47,10 @@
       <dynamics damping="0.3"/>
     </joint>
-    <link name="arm_elbow_link"/>
+    <!-- Khớp 3: elbow -->
+    <link name="arm_elbow_link">
+      <inertial><mass value="1.5"/></inertial>
+      <visual><geometry><box size="0.06 0.22 0.06"/></geometry><material name="orange"/></visual>
+      <collision><geometry><box size="0.06 0.22 0.06"/></geometry></collision>
+    </link>
     <joint name="arm_elbow_joint" type="revolute">
       <parent link="arm_shoulder_pitch_link"/>
@@ -41,5 +61,10 @@
       <dynamics damping="0.3"/>
     </joint>
-    <link name="ee_link"/>
+    <!-- EE -->
+    <link name="ee_link">
+      <inertial><mass value="0.5"/></inertial>
+      <visual><origin xyz="0 0 0.11"/><geometry><sphere radius="0.03"/></geometry><material name="orange"/></visual>
+      <collision><origin xyz="0 0 0.11"/><geometry><sphere radius="0.03"/></geometry></collision>
+    </link>
     <joint name="ee_fixed" type="fixed">
       <parent link="arm_elbow_link"/>

File: src/mobile_lift_arm/urdf/scissor_lift.xacro (robot description, xacro)
@@ -35,4 +35,7 @@
       <child link="lift_top_link"/>
     </joint>
+    <gazebo reference="lift_link">
+      <mu1>0.9</mu1><mu2>0.9</mu2>
+    </gazebo>
   </xacro:macro>
 </robot>
