Commit message: update

File: src/mobile_lift_arm/urdf/base_vehicle.xacro (robot description, xacro)
@@ -2,20 +2,20 @@
 <robot xmlns:xacro="http://www.ros.org/wiki/xacro" name="tricycle_base">
   <!-- Dimensions and parameters -->
-  <xacro:property name="BASE_LENGTH" value="0.6"/>   <!-- body length (x) -->
-  <xacro:property name="BASE_WIDTH"  value="0.4"/>   <!-- body width (y) -->
-  <xacro:property name="BASE_HEIGHT" value="0.1"/>  <!-- body height (z) -->
-  <xacro:property name="WHEEL_RADIUS" value="0.1"/>
-  <xacro:property name="WHEEL_THICK"  value="0.05"/>
-  <xacro:property name="CLEARANCE"    value="0.12"/> <!-- ground clearance -->
+  <xacro:property name="BASE_LENGTH" value="0.8"/>   <!-- body length (x) -->
+  <xacro:property name="BASE_WIDTH"  value="0.5"/>   <!-- body width (y) -->
+  <xacro:property name="BASE_HEIGHT" value="0.15"/>  <!-- body height (z) -->
+  <xacro:property name="WHEEL_RADIUS" value="0.15"/>
+  <xacro:property name="WHEEL_THICK"  value="0.08"/>
+  <xacro:property name="CLEARANCE"    value="0.18"/> <!-- ground clearance -->
   <!-- Tricycle specific parameters -->
-  <xacro:property name="REAR_WHEEL_SEPARATION" value="${BASE_WIDTH * 0.8}"/>  <!-- Distance between rear wheels -->
-  <xacro:property name="WHEELBASE" value="${BASE_LENGTH * 0.65}"/>            <!-- Distance from front to rear axle -->
+  <xacro:property name="REAR_WHEEL_SEPARATION" value="${BASE_WIDTH * 0.9}"/>  <!-- Distance between rear wheels -->
+  <xacro:property name="WHEELBASE" value="${BASE_LENGTH * 0.7}"/>            <!-- Distance from front to rear axle -->
   <xacro:property name="FRONT_WHEEL_OFFSET" value="${WHEELBASE/2}"/>          <!-- Front wheel position -->
   <xacro:property name="REAR_WHEEL_OFFSET" value="${-WHEELBASE/2}"/>          <!-- Rear wheels position -->
   <!-- Steering limits -->
-  <xacro:property name="MAX_STEER_ANGLE" value="0.7854"/>  <!-- 45 degrees in radians -->
+  <xacro:property name="MAX_STEER_ANGLE" value="1.0472"/>  <!-- 60 degrees in radians -->
   <!-- Mass properties -->
-  <xacro:property name="M_BASE"  value="20.0"/>
-  <xacro:property name="M_WHEEL" value="2.0"/>
+  <xacro:property name="M_BASE"  value="35.0"/>
+  <xacro:property name="M_WHEEL" value="3.5"/>
   <xacro:property name="M_STEER" value="1.0"/>  <!-- Steering assembly mass -->
   <!-- Inertia calculations -->
@@ -90,85 +90,85 @@
           <friction>
             <ode>
+              <mu>1.5</mu>
+              <mu2>1.5</mu2>
+            </ode>
+          </friction>
+        </surface>
+      </collision>
+    </link>
+    <!-- RIGHT REAR WHEEL -->
+    <link name="right_rear_wheel_link">
+      <inertial>
+        <origin xyz="0 0 0" rpy="0 0 0"/>
+        <mass value="${M_WHEEL}"/>
+        <inertia ixx="${Ixx_w}" iyy="${Iyy_w}" izz="${Izz_w}" ixy="0" ixz="0" iyz="0"/>
+      </inertial>
+      <visual>
+        <origin xyz="0 0 0" rpy="1.5708 0 0"/>
+        <geometry>
+          <cylinder radius="${WHEEL_RADIUS}" length="${WHEEL_THICK}"/>
+        </geometry>
+        <material name="wheel_black"/>
+      </visual>
+      <collision>
+        <origin xyz="0 0 0" rpy="1.5708 0 0"/>
+        <geometry>
+          <cylinder radius="${WHEEL_RADIUS}" length="${WHEEL_THICK}"/>
+        </geometry>
+        <surface>
+          <friction>
+            <ode>
+              <mu>1.5</mu>
+              <mu2>1.5</mu2>
+            </ode>
+          </friction>
+        </surface>
+      </collision>
+    </link>
+    <!-- FRONT STEERING ASSEMBLY -->
+    <link name="front_steer_link">
+      <inertial>
+        <origin xyz="0 0 0" rpy="0 0 0"/>
+        <mass value="${M_STEER}"/>
+        <inertia ixx="${Ixx_s}" iyy="${Iyy_s}" izz="${Izz_s}" ixy="0" ixz="0" iyz="0"/>
+      </inertial>
+      <visual>
+        <origin xyz="0 0 0" rpy="0 0 0"/>
+        <geometry>
+          <cylinder radius="0.02" length="0.1"/>
+        </geometry>
+        <material name="steer_red"><color rgba="0.8 0.1 0.1 1"/></material>
+      </visual>
+      <collision>
+        <origin xyz="0 0 0" rpy="0 0 0"/>
+        <geometry>
+          <cylinder radius="0.02" length="0.1"/>
+        </geometry>
+      </collision>
+    </link>
+    <!-- FRONT WHEEL -->
+    <link name="front_wheel_link">
+      <inertial>
+        <origin xyz="0 0 0" rpy="0 0 0"/>
+        <mass value="${M_WHEEL}"/>
+        <inertia ixx="${Ixx_w}" iyy="${Iyy_w}" izz="${Izz_w}" ixy="0" ixz="0" iyz="0"/>
+      </inertial>
+      <visual>
+        <origin xyz="0 0 0" rpy="1.5708 0 0"/>
+        <geometry>
+          <cylinder radius="${WHEEL_RADIUS}" length="${WHEEL_THICK}"/>
+        </geometry>
+        <material name="wheel_black"/>
+      </visual>
+      <collision>
+        <origin xyz="0 0 0" rpy="1.5708 0 0"/>
+        <geometry>
+          <cylinder radius="${WHEEL_RADIUS}" length="${WHEEL_THICK}"/>
+        </geometry>
+        <surface>
+          <friction>
+            <ode>
               <mu>1.2</mu>
               <mu2>1.2</mu2>
-            </ode>
-          </friction>
-        </surface>
-      </collision>
-    </link>
-    <!-- RIGHT REAR WHEEL -->
-    <link name="right_rear_wheel_link">
-      <inertial>
-        <origin xyz="0 0 0" rpy="0 0 0"/>
-        <mass value="${M_WHEEL}"/>
-        <inertia ixx="${Ixx_w}" iyy="${Iyy_w}" izz="${Izz_w}" ixy="0" ixz="0" iyz="0"/>
-      </inertial>
-      <visual>
-        <origin xyz="0 0 0" rpy="1.5708 0 0"/>
-        <geometry>
-          <cylinder radius="${WHEEL_RADIUS}" length="${WHEEL_THICK}"/>
-        </geometry>
-        <material name="wheel_black"/>
-      </visual>
-      <collision>
-        <origin xyz="0 0 0" rpy="1.5708 0 0"/>
-        <geometry>
-          <cylinder radius="${WHEEL_RADIUS}" length="${WHEEL_THICK}"/>
-        </geometry>
-        <surface>
-          <friction>
-            <ode>
-              <mu>1.2</mu>
-              <mu2>1.2</mu2>
-            </ode>
-          </friction>
-        </surface>
-      </collision>
-    </link>
-    <!-- FRONT STEERING ASSEMBLY -->
-    <link name="front_steer_link">
-      <inertial>
-        <origin xyz="0 0 0" rpy="0 0 0"/>
-        <mass value="${M_STEER}"/>
-        <inertia ixx="${Ixx_s}" iyy="${Iyy_s}" izz="${Izz_s}" ixy="0" ixz="0" iyz="0"/>
-      </inertial>
-      <visual>
-        <origin xyz="0 0 0" rpy="0 0 0"/>
-        <geometry>
-          <cylinder radius="0.02" length="0.1"/>
-        </geometry>
-        <material name="steer_red"><color rgba="0.8 0.1 0.1 1"/></material>
-      </visual>
-      <collision>
-        <origin xyz="0 0 0" rpy="0 0 0"/>
-        <geometry>
-          <cylinder radius="0.02" length="0.1"/>
-        </geometry>
-      </collision>
-    </link>
-    <!-- FRONT WHEEL -->
-    <link name="front_wheel_link">
-      <inertial>
-        <origin xyz="0 0 0" rpy="0 0 0"/>
-        <mass value="${M_WHEEL}"/>
-        <inertia ixx="${Ixx_w}" iyy="${Iyy_w}" izz="${Izz_w}" ixy="0" ixz="0" iyz="0"/>
-      </inertial>
-      <visual>
-        <origin xyz="0 0 0" rpy="1.5708 0 0"/>
-        <geometry>
-          <cylinder radius="${WHEEL_RADIUS}" length="${WHEEL_THICK}"/>
-        </geometry>
-        <material name="wheel_black"/>
-      </visual>
-      <collision>
-        <origin xyz="0 0 0" rpy="1.5708 0 0"/>
-        <geometry>
-          <cylinder radius="${WHEEL_RADIUS}" length="${WHEEL_THICK}"/>
-        </geometry>
-        <surface>
-          <friction>
-            <ode>
-              <mu>1.0</mu>
-              <mu2>1.0</mu2>
             </ode>
           </friction>
@@ -180,5 +180,5 @@
       <parent link="base_link"/>
       <child  link="left_rear_wheel_link"/>
-      <origin xyz="${REAR_WHEEL_OFFSET} ${REAR_WHEEL_SEPARATION/2} ${WHEEL_RADIUS + CLEARANCE}" rpy="0 0 0"/>
+      <origin xyz="${REAR_WHEEL_OFFSET} ${REAR_WHEEL_SEPARATION/2} -${BASE_HEIGHT/2 + CLEARANCE - WHEEL_RADIUS}" rpy="0 0 0"/>
       <axis xyz="0 1 0"/>
       <limit effort="15" velocity="25"/>
@@ -188,5 +188,5 @@
       <parent link="base_link"/>
       <child  link="right_rear_wheel_link"/>
-      <origin xyz="${REAR_WHEEL_OFFSET} -${REAR_WHEEL_SEPARATION/2} ${WHEEL_RADIUS + CLEARANCE}" rpy="0 0 0"/>
+      <origin xyz="${REAR_WHEEL_OFFSET} -${REAR_WHEEL_SEPARATION/2} -${BASE_HEIGHT/2 + CLEARANCE - WHEEL_RADIUS}" rpy="0 0 0"/>
       <axis xyz="0 1 0"/>
       <limit effort="15" velocity="25"/>
@@ -197,5 +197,5 @@
       <parent link="base_link"/>
       <child  link="front_steer_link"/>
-      <origin xyz="${FRONT_WHEEL_OFFSET} 0 ${WHEEL_RADIUS + CLEARANCE}" rpy="0 0 0"/>
+      <origin xyz="${FRONT_WHEEL_OFFSET} 0 -${BASE_HEIGHT/2 + CLEARANCE - WHEEL_RADIUS}" rpy="0 0 0"/>
       <axis xyz="0 0 1"/>
       <limit lower="-${MAX_STEER_ANGLE}" upper="${MAX_STEER_ANGLE}" effort="10" velocity="2"/>
