Commit message: add robot arm 6 DOF

File: src/mobile_lift_arm/urdf/mobile_lift_arm.urdf.xacro (robot description, xacro)
@@ -36,18 +36,28 @@
       <state_interface name="velocity"/>
     </joint>
+    <!-- arm 6DOF -->
     <joint name="arm_shoulder_yaw_joint">
       <command_interface name="position"/>
-      <state_interface name="position"/>
-      <state_interface name="velocity"/>
+      <state_interface name="position"/><state_interface name="velocity"/>
     </joint>
     <joint name="arm_shoulder_pitch_joint">
       <command_interface name="position"/>
-      <state_interface name="position"/>
-      <state_interface name="velocity"/>
+      <state_interface name="position"/><state_interface name="velocity"/>
     </joint>
-    <joint name="arm_elbow_joint">
+    <joint name="arm_shoulder_roll_joint">
       <command_interface name="position"/>
-      <state_interface name="position"/>
-      <state_interface name="velocity"/>
+      <state_interface name="position"/><state_interface name="velocity"/>
+    </joint>
+    <joint name="arm_elbow_pitch_joint">
+      <command_interface name="position"/>
+      <state_interface name="position"/><state_interface name="velocity"/>
+    </joint>
+    <joint name="arm_wrist_pitch_joint">
+      <command_interface name="position"/>
+      <state_interface name="position"/><state_interface name="velocity"/>
+    </joint>
+    <joint name="arm_wrist_roll_joint">
+      <command_interface name="position"/>
+      <state_interface name="position"/><state_interface name="velocity"/>
     </joint>
   </ros2_control>

File: src/mobile_lift_arm/urdf/robot_arm.xacro (robot description, xacro)
@@ -1,15 +1,21 @@
 <?xml version="1.0"?>
 <robot xmlns:xacro="http://www.ros.org/wiki/xacro">
+  <!-- Arm 6-DOF with simple geometry and proper inertials -->
   <xacro:macro name="robot_arm" params="parent">
+    <!-- Base stub mounted to parent -->
     <link name="arm_base_link">
-      <inertial><mass value="3"/><inertia ixx="0.03" iyy="0.03" izz="0.03" ixy="0" ixz="0" iyz="0"/></inertial>
-      <visual>
-        <origin xyz="0 0 0.05" rpy="0 0 0"/>
-        <geometry><cylinder radius="0.06" length="0.1"/></geometry>
+      <inertial>
+        <origin xyz="0 0 0.05" rpy="0 0 0"/>
+        <mass value="3.0"/>
+        <inertia ixx="0.03" ixy="0" ixz="0" iyy="0.03" iyz="0" izz="0.03"/>
+      </inertial>
+      <visual>
+        <origin xyz="0 0 0.05" rpy="0 0 0"/>
+        <geometry><cylinder radius="0.06" length="0.10"/></geometry>
         <material name="orange"><color rgba="0.9 0.5 0.2 1"/></material>
       </visual>
       <collision>
         <origin xyz="0 0 0.05" rpy="0 0 0"/>
-        <geometry><cylinder radius="0.06" length="0.1"/></geometry>
+        <geometry><cylinder radius="0.06" length="0.10"/></geometry>
       </collision>
     </link>
@@ -17,6 +23,23 @@
       <parent link="${parent}"/>
       <child link="arm_base_link"/>
-    </joint>
-    <link name="arm_shoulder_yaw_link"/>
+      <origin xyz="0 0 0" rpy="0 0 0"/>
+    </joint>
+    <!-- J1: Shoulder Yaw (Z) -->
+    <link name="arm_shoulder_yaw_link">
+      <inertial>
+        <origin xyz="0 0 0.08" rpy="0 0 0"/>
+        <mass value="2.0"/>
+        <inertia ixx="0.02" ixy="0" ixz="0" iyy="0.02" iyz="0" izz="0.02"/>
+      </inertial>
+      <visual>
+        <origin xyz="0 0 0.08" rpy="0 0 0"/>
+        <geometry><box size="0.08 0.08 0.16"/></geometry>
+        <material name="orange"/>
+      </visual>
+      <collision>
+        <origin xyz="0 0 0.08" rpy="0 0 0"/>
+        <geometry><box size="0.08 0.08 0.16"/></geometry>
+      </collision>
+    </link>
     <joint name="arm_shoulder_yaw_joint" type="revolute">
       <parent link="arm_base_link"/>
@@ -24,30 +47,153 @@
       <origin xyz="0 0 0.07" rpy="0 0 0"/>
       <axis xyz="0 0 1"/>
-      <limit lower="-3.14" upper="3.14" effort="30" velocity="1.5"/>
-      <dynamics damping="0.3"/>
-    </joint>
-    <link name="arm_shoulder_pitch_link"/>
+      <limit lower="-3.14" upper="3.14" effort="40" velocity="1.5"/>
+      <dynamics damping="0.3" friction="0.1"/>
+    </joint>
+    <!-- J2: Shoulder Pitch (Y), link length ~0.25 -->
+    <link name="arm_shoulder_pitch_link">
+      <inertial>
+        <origin xyz="0 0 0.125" rpy="0 0 0"/>
+        <mass value="2.0"/>
+        <inertia ixx="0.02" ixy="0" ixz="0" iyy="0.02" iyz="0" izz="0.02"/>
+      </inertial>
+      <visual>
+        <origin xyz="0 0 0.125" rpy="0 0 0"/>
+        <geometry><box size="0.08 0.25 0.08"/></geometry>
+        <material name="orange"/>
+      </visual>
+      <collision>
+        <origin xyz="0 0 0.125" rpy="0 0 0"/>
+        <geometry><box size="0.08 0.25 0.08"/></geometry>
+      </collision>
+    </link>
     <joint name="arm_shoulder_pitch_joint" type="revolute">
       <parent link="arm_shoulder_yaw_link"/>
       <child link="arm_shoulder_pitch_link"/>
-      <origin xyz="0 0 0.1" rpy="0 0 0"/>
+      <origin xyz="0 0 0.12" rpy="0 0 0"/>
       <axis xyz="0 1 0"/>
-      <limit lower="-1.57" upper="1.57" effort="30" velocity="1.2"/>
-      <dynamics damping="0.3"/>
-    </joint>
-    <link name="arm_elbow_link"/>
-    <joint name="arm_elbow_joint" type="revolute">
+      <limit lower="-1.8" upper="1.8" effort="40" velocity="1.2"/>
+      <dynamics damping="0.3" friction="0.1"/>
+    </joint>
+    <!-- J3: Shoulder Roll (X) -->
+    <link name="arm_shoulder_roll_link">
+      <inertial>
+        <origin xyz="0 0 0.06" rpy="0 0 0"/>
+        <mass value="1.8"/>
+        <inertia ixx="0.018" ixy="0" ixz="0" iyy="0.018" iyz="0" izz="0.018"/>
+      </inertial>
+      <visual>
+        <origin xyz="0 0 0.06" rpy="0 0 0"/>
+        <geometry><box size="0.08 0.12 0.12"/></geometry>
+        <material name="orange"/>
+      </visual>
+      <collision>
+        <origin xyz="0 0 0.06" rpy="0 0 0"/>
+        <geometry><box size="0.08 0.12 0.12"/></geometry>
+      </collision>
+    </link>
+    <joint name="arm_shoulder_roll_joint" type="revolute">
       <parent link="arm_shoulder_pitch_link"/>
+      <child link="arm_shoulder_roll_link"/>
+      <origin xyz="0 0 0.20" rpy="0 0 0"/>
+      <axis xyz="1 0 0"/>
+      <limit lower="-2.8" upper="2.8" effort="30" velocity="1.2"/>
+      <dynamics damping="0.3" friction="0.1"/>
+    </joint>
+    <!-- J4: Elbow Pitch (Y), forearm length ~0.22 -->
+    <link name="arm_elbow_link">
+      <inertial>
+        <origin xyz="0 0 0.11" rpy="0 0 0"/>
+        <mass value="1.6"/>
+        <inertia ixx="0.016" ixy="0" ixz="0" iyy="0.016" iyz="0" izz="0.016"/>
+      </inertial>
+      <visual>
+        <origin xyz="0 0 0.11" rpy="0 0 0"/>
+        <geometry><box size="0.06 0.22 0.06"/></geometry>
+        <material name="orange"/>
+      </visual>
+      <collision>
+        <origin xyz="0 0 0.11" rpy="0 0 0"/>
+        <geometry><box size="0.06 0.22 0.06"/></geometry>
+      </collision>
+    </link>
+    <joint name="arm_elbow_pitch_joint" type="revolute">
+      <parent link="arm_shoulder_roll_link"/>
       <child link="arm_elbow_link"/>
-      <origin xyz="0 0 0.125" rpy="0 0 0"/>
+      <origin xyz="0 0 0.06" rpy="0 0 0"/>
       <axis xyz="0 1 0"/>
-      <limit lower="-1.57" upper="1.57" effort="20" velocity="1.2"/>
-      <dynamics damping="0.3"/>
-    </joint>
-    <link name="ee_link"/>
+      <limit lower="-2.6" upper="2.6" effort="25" velocity="1.2"/>
+      <dynamics damping="0.25" friction="0.08"/>
+    </joint>
+    <!-- J5: Wrist Pitch (Y) -->
+    <link name="arm_wrist_pitch_link">
+      <inertial>
+        <origin xyz="0 0 0.05" rpy="0 0 0"/>
+        <mass value="1.0"/>
+        <inertia ixx="0.01" ixy="0" ixz="0" iyy="0.01" iyz="0" izz="0.01"/>
+      </inertial>
+      <visual>
+        <origin xyz="0 0 0.05" rpy="0 0 0"/>
+        <geometry><box size="0.05 0.10 0.05"/></geometry>
+        <material name="orange"/>
+      </visual>
+      <collision>
+        <origin xyz="0 0 0.05" rpy="0 0 0"/>
+        <geometry><box size="0.05 0.10 0.05"/></geometry>
+      </collision>
+    </link>
+    <joint name="arm_wrist_pitch_joint" type="revolute">
+      <parent link="arm_elbow_link"/>
+      <child link="arm_wrist_pitch_link"/>
+      <origin xyz="0 0 0.20" rpy="0 0 0"/>
+      <axis xyz="0 1 0"/>
+      <limit lower="-2.2" upper="2.2" effort="20" velocity="1.5"/>
+      <dynamics damping="0.2" friction="0.05"/>
+    </joint>
+    <!-- J6: Wrist Roll (Z) -->
+    <link name="arm_wrist_roll_link">
+      <inertial>
+        <origin xyz="0 0 0.03" rpy="0 0 0"/>
+        <mass value="0.8"/>
+        <inertia ixx="0.008" ixy="0" ixz="0" iyy="0.008" iyz="0" izz="0.008"/>
+      </inertial>
+      <visual>
+        <origin xyz="0 0 0.03" rpy="0 0 0"/>
+        <geometry><cylinder radius="0.035" length="0.06"/></geometry>
+        <material name="orange"/>
+      </visual>
+      <collision>
+        <origin xyz="0 0 0.03" rpy="0 0 0"/>
+        <geometry><cylinder radius="0.035" length="0.06"/></geometry>
+      </collision>
+    </link>
+    <joint name="arm_wrist_roll_joint" type="revolute">
+      <parent link="arm_wrist_pitch_link"/>
+      <child link="arm_wrist_roll_link"/>
+      <origin xyz="0 0 0.10" rpy="0 0 0"/>
+      <axis xyz="0 0 1"/>
+      <limit lower="-3.14" upper="3.14" effort="15" velocity="1.8"/>
+      <dynamics damping="0.15" friction="0.04"/>
+    </joint>
+    <!-- End-effector (dummy) -->
+    <link name="ee_link">
+      <inertial>
+        <origin xyz="0 0 0.03" rpy="0 0 0"/>
+        <mass value="0.3"/>
+        <inertia ixx="0.003" ixy="0" ixz="0" iyy="0.003" iyz="0" izz="0.003"/>
+      </inertial>
+      <visual>
+        <origin xyz="0 0 0.03" rpy="0 0 0"/>
+        <geometry><sphere radius="0.03"/></geometry>
+        <material name="orange"/>
+      </visual>
+      <collision>
+        <origin xyz="0 0 0.03" rpy="0 0 0"/>
+        <geometry><sphere radius="0.03"/></geometry>
+      </collision>
+    </link>
     <joint name="ee_fixed" type="fixed">
-      <parent link="arm_elbow_link"/>
+      <parent link="arm_wrist_roll_link"/>
       <child link="ee_link"/>
-      <origin xyz="0 0 0.11" rpy="0 0 0"/>
+      <origin xyz="0 0 0.06" rpy="0 0 0"/>
     </joint>
   </xacro:macro>

Commit message: add arm 6dof

File: src/mobile_lift_arm/urdf/mobile_lift_arm.urdf.xacro (robot description, xacro)
@@ -1,64 +1,20 @@
 <?xml version="1.0"?>
-<robot name="mobile_lift_arm" xmlns:xacro="http://www.ros.org/wiki/xacro">
+<robot name="mobile_lift_arm"
+  xmlns:xi="http://www.w3.org/2001/XInclude" xmlns:xacro="http://www.ros.org/wiki/xacro">
   <xacro:include filename="$(find mobile_lift_arm)/urdf/base_vehicle.xacro"/>
   <xacro:include filename="$(find mobile_lift_arm)/urdf/scissor_lift.xacro"/>
   <xacro:include filename="$(find mobile_lift_arm)/urdf/robot_arm.xacro"/>
+  <xacro:include filename="$(find mobile_lift_arm)/urdf/robot_arm_6dof_wrapper.xacro"/>
   <!-- Base -->
   <xacro:base_vehicle/>
   <!-- Lift gắn trên base_link -->
   <xacro:scissor_lift parent="base_link"/>
-  <!-- Arm gắn trên lift_top_link -->
-  <xacro:robot_arm parent="lift_top_link"/>
-  <!-- Gazebo ros2_control -->
-  <gazebo>
-    <plugin name="gazebo_ros2_control" filename="libgazebo_ros2_control.so">
-      <!-- ép namespace khớp với -entity -->
-      <robotNamespace>/mobile_lift_arm</robotNamespace>
-      <parameters>$(find mobile_lift_arm)/config/ros2_controllers.yaml</parameters>
-    </plugin>
-  </gazebo>
-  <!-- ros2_control -->
-  <ros2_control name="GazeboSystem" type="system">
-    <hardware><plugin>gazebo_ros2_control/GazeboSystem</plugin></hardware>
-    <joint name="left_wheel_joint">
-      <command_interface name="velocity"/>
-      <state_interface name="position"/>
-      <state_interface name="velocity"/>
-    </joint>
-    <joint name="right_wheel_joint">
-      <command_interface name="velocity"/>
-      <state_interface name="position"/>
-      <state_interface name="velocity"/>
-    </joint>
-    <joint name="lift_joint">
-      <command_interface name="position"/>
-      <state_interface name="position"/>
-      <state_interface name="velocity"/>
-    </joint>
-    <!-- arm 6DOF -->
-    <joint name="arm_shoulder_yaw_joint">
-      <command_interface name="position"/>
-      <state_interface name="position"/><state_interface name="velocity"/>
-    </joint>
-    <joint name="arm_shoulder_pitch_joint">
-      <command_interface name="position"/>
-      <state_interface name="position"/><state_interface name="velocity"/>
-    </joint>
-    <joint name="arm_shoulder_roll_joint">
-      <command_interface name="position"/>
-      <state_interface name="position"/><state_interface name="velocity"/>
-    </joint>
-    <joint name="arm_elbow_pitch_joint">
-      <command_interface name="position"/>
-      <state_interface name="position"/><state_interface name="velocity"/>
-    </joint>
-    <joint name="arm_wrist_pitch_joint">
-      <command_interface name="position"/>
-      <state_interface name="position"/><state_interface name="velocity"/>
-    </joint>
-    <joint name="arm_wrist_roll_joint">
-      <command_interface name="position"/>
-      <state_interface name="position"/><state_interface name="velocity"/>
-    </joint>
-  </ros2_control>
+  <!-- arm joints conditional -->
+  <joint name="arm_j1"><command_interface name="position"/><state_interface name="position"/><state_interface name="velocity"/></joint>
+  <joint name="arm_j2"><command_interface name="position"/><state_interface name="position"/><state_interface name="velocity"/></joint>
+  <joint name="arm_j3"><command_interface name="position"/><state_interface name="position"/><state_interface name="velocity"/></joint>
+  <joint name="arm_j4"><command_interface name="position"/><state_interface name="position"/><state_interface name="velocity"/></joint>
+  <joint name="arm_j5"><command_interface name="position"/><state_interface name="position"/><state_interface name="velocity"/></joint>
+  <joint name="arm_j6"><command_interface name="position"/><state_interface name="position"/><state_interface name="velocity"/></joint>
+</ros2_control>
 </robot>
