Commit message: update

File: src/mobile_lift_arm/urdf/mobile_lift_arm.urdf.xacro (robot description, xacro)
@@ -5,16 +5,9 @@
   <xacro:include filename="$(find mobile_lift_arm)/urdf/scissor_lift.xacro"/>
   <xacro:include filename="$(find mobile_lift_arm)/urdf/robot_arm.xacro"/>
-  <xacro:include filename="$(find mobile_lift_arm)/urdf/robot_arm_6dof_wrapper.xacro"/>
-  <!-- Base -->
+<!-- Base -->
   <xacro:base_vehicle/>
   <!-- Lift gắn trên base_link -->
   <xacro:scissor_lift parent="base_link"/>
   <!-- arm joints conditional -->
-  <joint name="arm_j1"><command_interface name="position"/><state_interface name="position"/><state_interface name="velocity"/></joint>
-  <joint name="arm_j2"><command_interface name="position"/><state_interface name="position"/><state_interface name="velocity"/></joint>
-  <joint name="arm_j3"><command_interface name="position"/><state_interface name="position"/><state_interface name="velocity"/></joint>
-  <joint name="arm_j4"><command_interface name="position"/><state_interface name="position"/><state_interface name="velocity"/></joint>
-  <joint name="arm_j5"><command_interface name="position"/><state_interface name="position"/><state_interface name="velocity"/></joint>
-  <joint name="arm_j6"><command_interface name="position"/><state_interface name="position"/><state_interface name="velocity"/></joint>
 </ros2_control>
 </robot>

File: src/mobile_lift_arm/urdf/robot_arm.xacro (robot description, xacro)
@@ -1,200 +1,302 @@
 <?xml version="1.0"?>
 <robot xmlns:xacro="http://www.ros.org/wiki/xacro">
-  <!-- Arm 6-DOF with simple geometry and proper inertials -->
+  <!-- 6-DOF arm as a single reusable macro -->
   <xacro:macro name="robot_arm" params="parent">
-    <!-- Base stub mounted to parent -->
-    <link name="arm_base_link">
-      <inertial>
-        <origin xyz="0 0 0.05" rpy="0 0 0"/>
-        <mass value="3.0"/>
-        <inertia ixx="0.03" ixy="0" ixz="0" iyy="0.03" iyz="0" izz="0.03"/>
-      </inertial>
-      <visual>
-        <origin xyz="0 0 0.05" rpy="0 0 0"/>
-        <geometry><cylinder radius="0.06" length="0.10"/></geometry>
-        <material name="orange"><color rgba="0.9 0.5 0.2 1"/></material>
-      </visual>
-      <collision>
-        <origin xyz="0 0 0.05" rpy="0 0 0"/>
-        <geometry><cylinder radius="0.06" length="0.10"/></geometry>
-      </collision>
-    </link>
-    <joint name="arm_base_fixed" type="fixed">
-      <parent link="${parent}"/>
+<!-- Define gray color -->
+  <material name="gray">
+   <color rgba="0.75 0.75 0.75 1.0"/>
+  </material>
+<!-- Define silver color -->
+<material name="silver">
+    <!-- <color rgba="0.75 0.75 0.75 1.0"/> -->
+    <color rgba="0.9 0.9 0.98 1.0"/>
+</material>
+<!-- Fixed Link -->
+<link name="arm_base_link"></link>
+<!-- Fixed Joint -->
+<joint name="arm_j0" type="fixed">
+    <origin xyz="0.0 0.0 0.0" rpy="0.0 0.0 0.0"/>
+    <parent link="arm_base_link"/>
+    <child link="arm_l0"/>
+    <axis xyz="0.0 0.0 0.0"/>
+    <limit lower="0.0" upper="0.0" effort="0.0" velocity="0.0"/>
+</joint>
+<link name="arm_l0">
+    <inertial>
+			<origin xyz="0.0 0.0 25e-03" rpy="0 0 0"/>
+			<mass value="2e+00"/>
+			<inertia
+				ixx="9.3895308e-03" ixy="0.0" ixz="1.1882474e-03"
+				iyx="0.0" iyy="1.4207390e-02" iyz="9.2874266e-06"
+				izx="1.1882474e-04"  izy="9.2874266e-06"  izz="1.7661948e-02"/>
+	</inertial>
+    <visual>
+        <geometry>
+            <cylinder radius="0.1" length="0.05"/>
+        </geometry>
+        <origin xyz="0.0 0.0 0.0" rpy="0.0 0.0 0.0"/>
+        <material name="silver"/>
+    </visual>
+</link>
+<joint name="arm_j1" type="revolute">
+    <origin xyz="0.0 0.0 0.0" rpy="0.0 0.0 0.0"/>
+    <parent link="arm_l0"/>
+    <child link="arm_l1"/>
+    <axis xyz="0.0 0.0 1.0"/>
+    <limit lower="-${2*pi}" upper="${2*pi}" effort="0.0" velocity="0.0"/>
+</joint>
+<link name="arm_l1">
+     <inertial>
+			<origin xyz="0.0 0.0 +0.25" rpy="0 0 0"/>
+			<mass value="1e+00"/>
+			<inertia
+            ixx="1.3778118e-01" ixy="5.1395441e-06" ixz="2.1163457e-04"
+            iyx="5.1395441e-06" iyy="1.3826689e-01" iyz="1.1751288e-02"
+            izx="2.1163457e-04" izy="1.1751288e-02" izz="3.5020186e-02"/>
+	</inertial>
+    <visual>
+        <geometry>
+            <cylinder radius="0.03" length="0.2"/>
+        </geometry>
+        <origin xyz="0.0 0.0 0.1" rpy="0.0 0.0 0.0"/>
+        <material name="silver"/>
+    </visual>
+    <!-- Add a sphere to create a curved joint -->
+    <visual>
+      <geometry>
+        <sphere radius="0.035"/>
+      </geometry>
+      <origin xyz="0.0 0.0 0.2" rpy="0.0 0.0 0.0"/>
+      <material name="gray"/>
+    </visual>
+</link>
+<!-- Dummy Joint -->
+<joint name="arm_j_dummy_1_2" type="fixed">
+    <origin xyz="0.0 0.0 0.2" rpy="0.0 0.0 0.0"/>
+    <parent link="arm_l1"/>
+    <child link="arm_l2"/>
+</joint>
+<link name="arm_l2">
+     <inertial>
+			<origin xyz="0.25 0.0 0.0" rpy="0 0 0"/>
+			<mass value="1e+00"/>
+			<inertia
+				ixx="3.0406895e-01" ixy="5.6383979e-04" ixz="4.4113010e-01"
+				iyx="5.6383979e-04" iyy="1.9934350e+00" iyz="1.2111129e-06"
+				izx="4.4113010e-01" izy="1.2111129e-06" izz="1.7471456e+00"/>
+	</inertial>
+    <visual>
+        <geometry>
+            <cylinder radius="0.03" length="0.25"/>
+        </geometry>
+        <origin xyz="0.125 0.0 0.0" rpy="0.0 ${pi/2} 0.0"/>
+        <material name="silver"/>
+    </visual>
+    <!-- Add a sphere to create a curved joint -->
+    <visual>
+      <geometry>
+        <sphere radius="0.035"/>
+      </geometry>
+      <origin xyz="0.25 0.0 0.0" rpy="0.0 0.0 0.0"/>
+      <material name="gray"/>
+    </visual>
+</link>
+<joint name="arm_j2" type="revolute">
+    <origin xyz="0.25 0.0 0.0" rpy="0.0 ${pi/2} 0.0"/>
+    <parent link="arm_l2"/>
+    <child link="arm_l3"/>
+    <axis xyz="0.0 0.0 1.0"/>
+    <limit lower="${-pi/2}" upper="${pi/2}" effort="0.0" velocity="0.0"/>
+</joint>
+<link name="arm_l3">
+     <inertial>
+			<origin xyz="-0.15 0.0 0.0" rpy="0 0 0"/>
+			<mass value="3e+00"/>
+			<inertia
+				ixx="3.1982320e-02" ixy="-1.5528529e-05" ixz="-4.8994800e-05"
+				iyx="-1.5528529e-05" iyy="2.8261283e-02" iyz="7.1406845e-03"
+				izx="-4.8994800e-05" izy="7.1406845e-03" izz="8.8063347e-03"/>
+	</inertial>
+    <visual>
+        <geometry>
+            <cylinder radius="0.03" length="0.3"/>
+        </geometry>
+        <origin xyz="-0.15 0.0 0.0 " rpy="0.0  ${pi/2} 0.0"/>
+        <material name="silver"/>
+    </visual>
+    <!-- Add a sphere to create a curved joint -->
+    <visual>
+      <geometry>
+        <sphere radius="0.035"/>
+      </geometry>
+      <origin xyz="0.0 0.0 0.0" rpy="0.0 0.0 0.0"/>
+      <material name="gray"/>
+    </visual>
+</link>
+<joint name="arm_j3" type="revolute">
+    <origin xyz="-0.30 0.0 0.0" rpy="0.0 0.0 0.0"/>
+    <parent link="arm_l3"/>
+    <child link="arm_l4"/>
+    <axis xyz="0.0 0.0 1.0"/>
+    <limit lower="${-pi/2}" upper="${pi/2}" effort="0.0" velocity="0.0"/>
+</joint>
+<link name="arm_l4">
+     <inertial>
+			<origin xyz="0.0 0.0 -0.12" rpy="0 0 0"/>
+			<mass value="1e+00"/>
+			<inertia
+				ixx="3.0406895e-01" ixy="5.6383979e-04" ixz="4.4113010e-01"
+				iyx="5.6383979e-04" iyy="1.9934350e+00" iyz="1.2111129e-06"
+				izx="4.4113010e-01" izy="1.2111129e-06" izz="1.7471456e+00"/>
+	</inertial>
+    <visual>
+        <geometry>
+            <cylinder radius="0.03" length="0.24"/>
+        </geometry>
+        <origin xyz="0.0 0.0 -0.12" rpy="0.0 0.0 0.0"/>
+        <material name="silver"/>
+    </visual>
+    <!-- Add a sphere to create a curved joint -->
+    <visual>
+      <geometry>
+        <sphere radius="0.035"/>
+      </geometry>
+      <origin xyz="0.0 0.0 0.0" rpy="0.0 0.0 0.0"/>
+      <material name="gray"/>
+    </visual>
+</link>
+<!-- Dummy Joint -->
+<joint name="arm_j_dummy" type="fixed">
+    <origin xyz="0.0 0.0 -0.24" rpy="0.0 0.0 0.0"/>
+    <parent link="arm_l4"/>
+    <child link="arm_l5"/>
+</joint>
+<link name="arm_l5">
+     <inertial>
+			<origin xyz="-0.16 0.0 0.0" rpy="0.0 0.0 0.0"/>
+			<mass value="3e+00"/>
+			<inertia
+				ixx="1.3754675e-02" ixy="-1.5528630e-05" ixz="-2.8051809e-05"
+				iyx="-1.5528630e-05" iyy="9.9916676e-03" iyz="3.9023300e-03"
+				izx="-2.8051809e-05" izy="3.9023300e-03" izz="7.6137437e-03"/>
+	</inertial>
+    <visual>
+        <geometry>
+            <cylinder radius="0.03" length="0.32"/>
+        </geometry>
+        <origin xyz="-0.16 0.0 0.0 " rpy="0.0 ${pi/2} 0.0"/>
+        <material name="silver"/>
+    </visual>
+    <!-- Add a sphere to create a curved joint -->
+    <visual>
+      <geometry>
+        <sphere radius="0.035"/>
+      </geometry>
+      <origin xyz="0.0 0.0 0.0" rpy="0.0 0.0 0.0"/>
+      <material name="gray"/>
+    </visual>
+</link>
+<joint name="arm_j4" type="revolute">
+    <origin xyz="-0.32 0.0 0.0" rpy="0.0 0.0 0.0"/>
+    <parent link="arm_l5"/>
+    <child link="arm_l6"/>
+    <axis xyz="0.0 0.0 1.0"/>
+    <limit lower="${-pi/2}" upper="${pi/2}" effort="0.0" velocity="0.0"/>
+</joint>
+<link name="arm_l6">
+     <inertial>
+			 <origin xyz="0.0 0.0 0.125" rpy="0.0 0.0 0.0"/>
+			<mass value="1e+00"/>
+			<inertia
+				ixx="9.3016047e-04" ixy="-2.9405026e-07" ixz="1.0421409e-05"
+				iyx="-2.9405026e-07" iyy="9.5021553e-04" iyz="-1.7371494e-06"
+				izx="1.0421409e-05" izy="-1.7371494e-06" izz="8.4567154e-04"/>
+	</inertial>
+    <visual>
+        <geometry>
+            <cylinder radius="0.03" length="0.25"/>
+        </geometry>
+        <origin xyz="0.0 0.0 0.125" rpy="0.0 0.0 0.0"/>
+        <material name="silver"/>
+    </visual>
+    <!-- Add a sphere to create a curved joint -->
+    <visual>
+      <geometry>
+        <sphere radius="0.035"/>
+      </geometry>
+      <origin xyz="0.0 0.0 0.0" rpy="0.0 0.0 0.0"/>
+      <material name="gray"/>
+    </visual>
+</link>
+<joint name="arm_j5" type="revolute">
+    <origin xyz="0.0 0.0 0.25" rpy="0.0 ${-pi/2} ${2*pi}"/>
+    <parent link="arm_l6"/>
+    <child link="arm_le"/>
+    <axis xyz="0.0 0.0 1.0"/>
+    <limit lower="${-pi}" upper="${pi}" effort="0.0" velocity="0.0"/>
+</joint>
+<link name="arm_le">
+     <inertial>
+			 <origin xyz="0.0 0.0 0.09" rpy="0.0 0.0 0.0"/>
+			<mass value="1e+00"/>
+			<inertia
+				ixx="9.3016047e-04" ixy="-2.9405026e-07" ixz="1.0421409e-05"
+				iyx="-2.9405026e-07" iyy="9.5021553e-04" iyz="-1.7371494e-06"
+				izx="1.0421409e-05" izy="-1.7371494e-06" izz="8.4567154e-04"/>
+	</inertial>
+    <visual>
+        <geometry>
+            <cylinder radius="0.03" length="0.18"/>
+        </geometry>
+        <origin xyz="0.0 0.0 0.09" rpy="0.0 0.0 0.0"/>
+        <material name="silver"/>
+    </visual>
+    <!-- Add a sphere to create a curved joint -->
+    <visual>
+      <geometry>
+        <sphere radius="0.035"/>
+      </geometry>
+      <origin xyz="0.0 0.0 0.0" rpy="0.0 0.0 0.0"/>
+      <material name="gray"/>
+    </visual>
+</link>
+<joint name="arm_j6" type="revolute">
+    <origin xyz="0.0 0.0 0.18" rpy="0.0 ${pi/2} 0.0"/>
+    <parent link="arm_le"/>
+    <child link="arm_le_1"/>
+    <axis xyz="0.0 0.0 1.0"/>
+    <limit lower="-${2*pi}" upper="${2*pi}" effort="0.0" velocity="0.0"/>
+</joint>
+<link name="arm_le_1">
+     <inertial>
+			 <origin xyz="0.0 0.0 0.05" rpy="0.0 0.0 0.0"/>
+			<mass value="1e+00"/>
+			<inertia
+				ixx="9.3016047e-04" ixy="-2.9405026e-07" ixz="1.0421409e-05"
+				iyx="-2.9405026e-07" iyy="9.5021553e-04" iyz="-1.7371494e-06"
+				izx="1.0421409e-05" izy="-1.7371494e-06" izz="8.4567154e-04"/>
+	</inertial>
+    <visual>
+        <geometry>
+            <cylinder radius="0.03" length="0.1"/>
+        </geometry>
+        <origin xyz="0.0 0.0 0.05 " rpy="0.0 0.0 0.0"/>
+        <material name="gray"/>
+    </visual>
+    <!-- Add a sphere to create a curved joint -->
+    <visual>
+      <geometry>
+        <sphere radius="0.035"/>
+      </geometry>
+      <origin xyz="0.0 0.0 0.0" rpy="0.0 0.0 0.0"/>
+      <material name="gray"/>
+    </visual>
+</link>
+    <!-- Mount to parent (e.g., lift_top_link) -->
+    <joint name="arm_base_mount" type="fixed">
+      <parent link="{parent}"/>
       <child link="arm_base_link"/>
       <origin xyz="0 0 0" rpy="0 0 0"/>
     </joint>
-    <!-- J1: Shoulder Yaw (Z) -->
-    <link name="arm_shoulder_yaw_link">
-      <inertial>
-        <origin xyz="0 0 0.08" rpy="0 0 0"/>
-        <mass value="2.0"/>
-        <inertia ixx="0.02" ixy="0" ixz="0" iyy="0.02" iyz="0" izz="0.02"/>
-      </inertial>
-      <visual>
-        <origin xyz="0 0 0.08" rpy="0 0 0"/>
-        <geometry><box size="0.08 0.08 0.16"/></geometry>
-        <material name="orange"/>
-      </visual>
-      <collision>
-        <origin xyz="0 0 0.08" rpy="0 0 0"/>
-        <geometry><box size="0.08 0.08 0.16"/></geometry>
-      </collision>
-    </link>
-    <joint name="arm_shoulder_yaw_joint" type="revolute">
-      <parent link="arm_base_link"/>
-      <child link="arm_shoulder_yaw_link"/>
-      <origin xyz="0 0 0.07" rpy="0 0 0"/>
-      <axis xyz="0 0 1"/>
-      <limit lower="-3.14" upper="3.14" effort="40" velocity="1.5"/>
-      <dynamics damping="0.3" friction="0.1"/>
-    </joint>
-    <!-- J2: Shoulder Pitch (Y), link length ~0.25 -->
-    <link name="arm_shoulder_pitch_link">
-      <inertial>
-        <origin xyz="0 0 0.125" rpy="0 0 0"/>
-        <mass value="2.0"/>
-        <inertia ixx="0.02" ixy="0" ixz="0" iyy="0.02" iyz="0" izz="0.02"/>
-      </inertial>
-      <visual>
-        <origin xyz="0 0 0.125" rpy="0 0 0"/>
-        <geometry><box size="0.08 0.25 0.08"/></geometry>
-        <material name="orange"/>
-      </visual>
-      <collision>
-        <origin xyz="0 0 0.125" rpy="0 0 0"/>
-        <geometry><box size="0.08 0.25 0.08"/></geometry>
-      </collision>
-    </link>
-    <joint name="arm_shoulder_pitch_joint" type="revolute">
-      <parent link="arm_shoulder_yaw_link"/>
-      <child link="arm_shoulder_pitch_link"/>
-      <origin xyz="0 0 0.12" rpy="0 0 0"/>
-      <axis xyz="0 1 0"/>
-      <limit lower="-1.8" upper="1.8" effort="40" velocity="1.2"/>
-      <dynamics damping="0.3" friction="0.1"/>
-    </joint>
-    <!-- J3: Shoulder Roll (X) -->
-    <link name="arm_shoulder_roll_link">
-      <inertial>
-        <origin xyz="0 0 0.06" rpy="0 0 0"/>
-        <mass value="1.8"/>
-        <inertia ixx="0.018" ixy="0" ixz="0" iyy="0.018" iyz="0" izz="0.018"/>
-      </inertial>
-      <visual>
-        <origin xyz="0 0 0.06" rpy="0 0 0"/>
-        <geometry><box size="0.08 0.12 0.12"/></geometry>
-        <material name="orange"/>
-      </visual>
-      <collision>
-        <origin xyz="0 0 0.06" rpy="0 0 0"/>
-        <geometry><box size="0.08 0.12 0.12"/></geometry>
-      </collision>
-    </link>
-    <joint name="arm_shoulder_roll_joint" type="revolute">
-      <parent link="arm_shoulder_pitch_link"/>
-      <child link="arm_shoulder_roll_link"/>
-      <origin xyz="0 0 0.20" rpy="0 0 0"/>
-      <axis xyz="1 0 0"/>
-      <limit lower="-2.8" upper="2.8" effort="30" velocity="1.2"/>
-      <dynamics damping="0.3" friction="0.1"/>
-    </joint>
-    <!-- J4: Elbow Pitch (Y), forearm length ~0.22 -->
-    <link name="arm_elbow_link">
-      <inertial>
-        <origin xyz="0 0 0.11" rpy="0 0 0"/>
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
Commit message: Refactor: Use direct robot_arm macro instead of wrapper, complete ros2_control definition

File: src/mobile_lift_arm/urdf/mobile_lift_arm.urdf.xacro (robot description, xacro)
@@ -5,9 +5,96 @@
   <xacro:include filename="$(find mobile_lift_arm)/urdf/scissor_lift.xacro"/>
   <xacro:include filename="$(find mobile_lift_arm)/urdf/robot_arm.xacro"/>
-<!-- Base -->
+  <!-- Base -->
   <xacro:base_vehicle/>
   <!-- Lift gắn trên base_link -->
   <xacro:scissor_lift parent="base_link"/>
-  <!-- arm joints conditional -->
-</ros2_control>
+  <!-- Arm gắn trên lift_top_link -->
+  <xacro:robot_arm parent="lift_top_link"/>
+  <!-- ros2_control definition -->
+  <ros2_control name="mobile_lift_arm_system" type="system">
+    <hardware>
+      <plugin>gazebo_ros2_control/GazeboSystem</plugin>
+    </hardware>
+    <!-- Base wheels -->
+    <joint name="left_wheel_joint">
+      <command_interface name="velocity">
+        <param name="min">-10</param>
+        <param name="max">10</param>
+      </command_interface>
+      <state_interface name="position"/>
+      <state_interface name="velocity"/>
+    </joint>
+    <joint name="right_wheel_joint">
+      <command_interface name="velocity">
+        <param name="min">-10</param>
+        <param name="max">10</param>
+      </command_interface>
+      <state_interface name="position"/>
+      <state_interface name="velocity"/>
+    </joint>
+    <!-- Lift joint -->
+    <joint name="lift_joint">
+      <command_interface name="position">
+        <param name="min">0.0</param>
+        <param name="max">1.2</param>
+      </command_interface>
+      <state_interface name="position"/>
+      <state_interface name="velocity"/>
+    </joint>
+    <!-- Arm joints -->
+    <joint name="arm_j1">
+      <command_interface name="position">
+        <param name="min">-6.28</param>
+        <param name="max">6.28</param>
+      </command_interface>
+      <state_interface name="position"/>
+      <state_interface name="velocity"/>
+    </joint>
+    <joint name="arm_j2">
+      <command_interface name="position">
+        <param name="min">-1.57</param>
+        <param name="max">1.57</param>
+      </command_interface>
+      <state_interface name="position"/>
+      <state_interface name="velocity"/>
+    </joint>
+    <joint name="arm_j3">
+      <command_interface name="position">
+        <param name="min">-1.57</param>
+        <param name="max">1.57</param>
+      </command_interface>
+      <state_interface name="position"/>
+      <state_interface name="velocity"/>
+    </joint>
+    <joint name="arm_j4">
+      <command_interface name="position">
+        <param name="min">-1.57</param>
+        <param name="max">1.57</param>
+      </command_interface>
+      <state_interface name="position"/>
+      <state_interface name="velocity"/>
+    </joint>
+    <joint name="arm_j5">
+      <command_interface name="position">
+        <param name="min">-3.14</param>
+        <param name="max">3.14</param>
+      </command_interface>
+      <state_interface name="position"/>
+      <state_interface name="velocity"/>
+    </joint>
+    <joint name="arm_j6">
+      <command_interface name="position">
+        <param name="min">-6.28</param>
+        <param name="max">6.28</param>
+      </command_interface>
+      <state_interface name="position"/>
+      <state_interface name="velocity"/>
+    </joint>
+  </ros2_control>
+  <!-- Gazebo ros2_control plugin -->
+  <gazebo>
+    <plugin filename="libgazebo_ros2_control.so" name="gazebo_ros2_control">
+      <parameters>$(find mobile_lift_arm)/config/ros2_controllers.yaml</parameters>
+    </plugin>
+  </gazebo>
 </robot>

Commit message: Fix: Update ros2_control joint names to match arm joints

File: src/mobile_lift_arm/urdf/mobile_lift_arm.urdf.xacro (robot description, xacro)
@@ -43,5 +43,5 @@
     </joint>
     <!-- Arm joints -->
-    <joint name="arm_j1">
+    <joint name="arm_shoulder_yaw_joint">
       <command_interface name="position">
         <param name="min">-6.28</param>
@@ -51,5 +51,5 @@
       <state_interface name="velocity"/>
     </joint>
-    <joint name="arm_j2">
+    <joint name="arm_shoulder_pitch_joint">
       <command_interface name="position">
         <param name="min">-1.57</param>
@@ -59,5 +59,5 @@
       <state_interface name="velocity"/>
     </joint>
-    <joint name="arm_j3">
+    <joint name="arm_shoulder_roll_joint">
       <command_interface name="position">
         <param name="min">-1.57</param>
@@ -67,5 +67,5 @@
       <state_interface name="velocity"/>
     </joint>
-    <joint name="arm_j4">
+    <joint name="arm_elbow_pitch_joint">
       <command_interface name="position">
         <param name="min">-1.57</param>
@@ -75,5 +75,5 @@
       <state_interface name="velocity"/>
     </joint>
-    <joint name="arm_j5">
+    <joint name="arm_wrist_pitch_joint">
       <command_interface name="position">
         <param name="min">-3.14</param>
@@ -83,5 +83,5 @@
       <state_interface name="velocity"/>
     </joint>
-    <joint name="arm_j6">
+    <joint name="arm_wrist_roll_joint">
       <command_interface name="position">
         <param name="min">-6.28</param>

Commit message: some update

File: src/mobile_lift_arm/urdf/mobile_lift_arm.urdf.xacro (robot description, xacro)
@@ -11,22 +11,39 @@
   <!-- Arm mounted on lift_top_link -->
   <xacro:robot_arm parent="lift_top_link"/>
-  <!-- ros2_control definition -->
+  <!-- ros2_control definition - SỬA CHO ĐÚNG VỚI TRICYCLE -->
   <ros2_control name="mobile_lift_arm_system" type="system">
     <hardware>
       <plugin>gazebo_ros2_control/GazeboSystem</plugin>
     </hardware>
-    <!-- Base wheels -->
-    <joint name="left_wheel_joint">
+    <!-- Tricycle wheels - SỬA TÊN JOINTS -->
+    <joint name="front_wheel_joint">
       <command_interface name="velocity">
-        <param name="min">-10</param>
-        <param name="max">10</param>
+        <param name="min">-20</param>
+        <param name="max">20</param>
       </command_interface>
       <state_interface name="position"/>
       <state_interface name="velocity"/>
     </joint>
-    <joint name="right_wheel_joint">
+    <joint name="left_rear_wheel_joint">
       <command_interface name="velocity">
-        <param name="min">-10</param>
-        <param name="max">10</param>
+        <param name="min">-25</param>
+        <param name="max">25</param>
+      </command_interface>
+      <state_interface name="position"/>
+      <state_interface name="velocity"/>
+    </joint>
+    <joint name="right_rear_wheel_joint">
+      <command_interface name="velocity">
+        <param name="min">-25</param>
+        <param name="max">25</param>
+      </command_interface>
+      <state_interface name="position"/>
+      <state_interface name="velocity"/>
+    </joint>
+    <!-- Steering joint -->
+    <joint name="front_steer_joint">
+      <command_interface name="position">
+        <param name="min">-1.0472</param>
+        <param name="max">1.0472</param>
       </command_interface>
       <state_interface name="position"/>
@@ -42,5 +59,5 @@
       <state_interface name="velocity"/>
     </joint>
-    <!-- Arm joints -->
+    <!-- Arm joints - GIẢM EFFORT LIMIT -->
     <joint name="arm_shoulder_yaw_joint">
       <command_interface name="position">

File: src/mobile_lift_arm/urdf/robot_arm.xacro (robot description, xacro)
@@ -300,3 +300,14 @@
     </joint>
   </xacro:macro>
+  <gazebo reference="arm_base_link">
+  <collision_name>arm_base_collision</collision_name>
+  <surface>
+    <contact>
+      <ode>
+        <max_contacts>10</max_contacts>
+        <max_correcting_vel>0.1</max_correcting_vel>
+      </ode>
+    </contact>
+  </surface>
+</gazebo>
 </robot>
