Commit message: Replace with complete scissor lift mechanism from main branch

File: src/mobile_lift_arm/urdf/scissor_lift.xacro (robot description, xacro)
@@ -1,38 +1,174 @@
 <?xml version="1.0"?>
 <robot xmlns:xacro="http://www.ros.org/wiki/xacro">
-  <xacro:property name="LIFT_MIN" value="0.0"/>
-  <xacro:property name="LIFT_MAX" value="1.2"/>
-  <xacro:property name="TOP_XY"   value="0.5"/>
-  <xacro:property name="TOP_T"    value="0.05"/>
+  <!-- Include macros for inertia -->
+  <xacro:include filename="$(find mobile_lift_arm)/urdf/scissor_lift_macros.xacro"/>
+  <!-- Parameters -->
+  <xacro:property name="base_length" value="1.0"/>
+  <xacro:property name="base_width" value="0.8"/>
+  <xacro:property name="base_height" value="0.1"/>
+  <xacro:property name="scissor_arm_length" value="0.8"/>
+  <xacro:property name="scissor_arm_width" value="0.05"/>
+  <xacro:property name="scissor_arm_height" value="0.03"/>
+  <xacro:property name="platform_length" value="0.9"/>
+  <xacro:property name="platform_width" value="0.7"/>
+  <xacro:property name="platform_height" value="0.05"/>
   <xacro:macro name="scissor_lift" params="parent">
-    <link name="lift_link">
-      <inertial>
-        <origin xyz="0 0 ${TOP_T/2}" rpy="0 0 0"/>
-        <mass value="8.0"/>
-        <inertia ixx="0.08" ixy="0" ixz="0" iyy="0.08" iyz="0" izz="0.08"/>
-      </inertial>
+    <!-- Base Platform -->
+    <link name="lift_base">
       <visual>
-        <origin xyz="0 0 ${TOP_T/2}" rpy="0 0 0"/>
-        <geometry><box size="${TOP_XY} ${TOP_XY} ${TOP_T}"/></geometry>
-        <material name="blue"><color rgba="0.2 0.3 0.9 1"/></material>
+        <geometry><box size="${base_length} ${base_width} ${base_height}"/></geometry>
+        <material name="grey"><color rgba="0.5 0.5 0.5 1"/></material>
       </visual>
       <collision>
-        <origin xyz="0 0 ${TOP_T/2}" rpy="0 0 0"/>
-        <geometry><box size="${TOP_XY} ${TOP_XY} ${TOP_T}"/></geometry>
+        <geometry><box size="${base_length} ${base_width} ${base_height}"/></geometry>
       </collision>
+      <xacro:box_inertia m="20" x="${base_length}" y="${base_width}" z="${base_height}"/>
+    </link>
+    <joint name="lift_base_joint" type="fixed">
+      <parent link="${parent}"/>
+      <child link="lift_base"/>
+      <origin xyz="0 0 0.1" rpy="0 0 0"/>
+    </joint>
+    <!-- === Left Side === -->
+    <link name="lower_left_arm">
+      <visual>
+        <geometry><box size="${scissor_arm_length} ${scissor_arm_width} ${scissor_arm_height}"/></geometry>
+        <material name="blue"><color rgba="0 0 1 1"/></material>
+      </visual>
+      <collision>
+        <geometry><box size="${scissor_arm_length} ${scissor_arm_width} ${scissor_arm_height}"/></geometry>
+      </collision>
+      <xacro:box_inertia m="2" x="${scissor_arm_length}" y="${scissor_arm_width}" z="${scissor_arm_height}"/>
+    </link>
+    <joint name="lower_left_joint" type="revolute">
+      <parent link="lift_base"/>
+      <child link="lower_left_arm"/>
+      <origin xyz="-${scissor_arm_length/2} -${base_width/4} ${base_height/2}"/>
+      <axis xyz="0 1 0"/>
+      <limit lower="0.0" upper="1.57" effort="500" velocity="1.0"/>
+      <dynamics damping="2.0" friction="0.1"/>
+    </joint>
+    <link name="upper_left_arm">
+      <visual>
+        <geometry><box size="${scissor_arm_length} ${scissor_arm_width} ${scissor_arm_height}"/></geometry>
+        <material name="red"><color rgba="1 0 0 1"/></material>
+      </visual>
+      <collision>
+        <geometry><box size="${scissor_arm_length} ${scissor_arm_width} ${scissor_arm_height}"/></geometry>
+      </collision>
+      <xacro:box_inertia m="2" x="${scissor_arm_length}" y="${scissor_arm_width}" z="${scissor_arm_height}"/>
+    </link>
+    <joint name="left_cross_joint" type="revolute">
+      <parent link="lower_left_arm"/>
+      <child link="upper_left_arm"/>
+      <origin xyz="0 0 0" rpy="0 0 0"/>
+      <axis xyz="0 1 0"/>
+      <limit lower="-3.14" upper="3.14" effort="500" velocity="1.0"/>
+      <dynamics damping="2.0" friction="0.1"/>
+    </joint>
+    <!-- === Right Side === -->
+    <link name="lower_right_arm">
+      <visual>
+        <geometry><box size="${scissor_arm_length} ${scissor_arm_width} ${scissor_arm_height}"/></geometry>
+        <material name="blue"/>
+      </visual>
+      <collision>
+        <geometry><box size="${scissor_arm_length} ${scissor_arm_width} ${scissor_arm_height}"/></geometry>
+      </collision>
+      <xacro:box_inertia m="2" x="${scissor_arm_length}" y="${scissor_arm_width}" z="${scissor_arm_height}"/>
+    </link>
+    <joint name="lower_right_joint" type="revolute">
+      <parent link="lift_base"/>
+      <child link="lower_right_arm"/>
+      <origin xyz="-${scissor_arm_length/2} ${base_width/4} ${base_height/2}"/>
+      <axis xyz="0 1 0"/>
+      <limit lower="0.0" upper="1.57" effort="500" velocity="1.0"/>
+      <dynamics damping="2.0" friction="0.1"/>
+    </joint>
+    <link name="upper_right_arm">
+      <visual>
+        <geometry><box size="${scissor_arm_length} ${scissor_arm_width} ${scissor_arm_height}"/></geometry>
+        <material name="red"/>
+      </visual>
+      <collision>
+        <geometry><box size="${scissor_arm_length} ${scissor_arm_width} ${scissor_arm_height}"/></geometry>
+      </collision>
+      <xacro:box_inertia m="2" x="${scissor_arm_length}" y="${scissor_arm_width}" z="${scissor_arm_height}"/>
+    </link>
+    <joint name="right_cross_joint" type="revolute">
+      <parent link="lower_right_arm"/>
+      <child link="upper_right_arm"/>
+      <origin xyz="0 0 0" rpy="0 0 0"/>
+      <axis xyz="0 1 0"/>
+      <limit lower="-3.14" upper="3.14" effort="500" velocity="1.0"/>
+      <dynamics damping="2.0" friction="0.1"/>
+    </joint>
+    <!-- === Lift Platform === -->
+    <link name="lift_link">
+      <visual>
+        <geometry><box size="${platform_length} ${platform_width} ${platform_height}"/></geometry>
+        <material name="green"><color rgba="0 1 0 1"/></material>
+      </visual>
+      <collision>
+        <geometry><box size="${platform_length} ${platform_width} ${platform_height}"/></geometry>
+      </collision>
+      <xacro:box_inertia m="8" x="${platform_length}" y="${platform_width}" z="${platform_height}"/>
+    </link>
+    <joint name="platform_left_joint" type="revolute">
+      <parent link="upper_left_arm"/>
+      <child link="lift_link"/>
+      <origin xyz="${scissor_arm_length/2} 0 ${platform_height/2}"/>
+      <axis xyz="0 1 0"/>
+      <limit lower="-3.14" upper="3.14" effort="500" velocity="1.0"/>
+      <dynamics damping="2.0" friction="0.1"/>
+    </joint>
+    <joint name="platform_right_joint" type="fixed">
+      <parent link="lift_link"/>
+      <child link="upper_right_arm"/>
+      <origin xyz="0 -${base_width/2} 0" rpy="0 0 0"/>
+    </joint>
+    <!-- === Hydraulic Actuator === -->
+    <link name="piston_actuator_link">
+      <visual>
+        <geometry><cylinder length="0.1" radius="0.02"/></geometry>
+        <material name="black"><color rgba="0.2 0.2 0.2 1"/></material>
+      </visual>
+      <collision>
+        <geometry><cylinder length="0.1" radius="0.02"/></geometry>
+      </collision>
+      <xacro:cylinder_inertia m="1" r="0.02" l="0.1"/>
     </link>
     <joint name="lift_joint" type="prismatic">
-      <parent link="${parent}"/>
-      <child link="lift_link"/>
-      <origin xyz="0 0 0.15" rpy="0 0 0"/>
-      <axis xyz="0 0 1"/>
-      <limit lower="${LIFT_MIN}" upper="${LIFT_MAX}" effort="500" velocity="0.2"/>
-      <dynamics damping="5.0" friction="0.1"/>
+      <parent link="lift_base"/>
+      <child link="piston_actuator_link"/>
+      <origin xyz="0 0 ${base_height/2}" rpy="0 0 0"/>
+      <axis xyz="1 0 0"/>
+      <limit lower="-0.3" upper="0.3" effort="2000" velocity="0.2"/>
+      <dynamics damping="10.0" friction="0.2"/>
     </joint>
+    <joint name="actuator_to_left_arm" type="revolute">
+        <parent link="piston_actuator_link"/>
+        <child link="lower_left_arm"/>
+        <origin xyz="0 0 0" rpy="0 0 0"/>
+        <axis xyz="0 1 0"/>
+        <limit lower="-3.14" upper="3.14" effort="500" velocity="1.0"/>
+        <dynamics damping="2.0" friction="0.1"/>
+    </joint>
+    <!-- Top link for arm attachment -->
     <link name="lift_top_link"/>
     <joint name="lift_top_fixed" type="fixed">
       <parent link="lift_link"/>
       <child link="lift_top_link"/>
+      <origin xyz="0 0 ${platform_height/2}" rpy="0 0 0"/>
     </joint>
+    <!-- Gazebo materials -->
+    <gazebo reference="lift_base"><material>Gazebo/Grey</material></gazebo>
+    <gazebo reference="lift_link"><material>Gazebo/Green</material></gazebo>
+    <gazebo reference="lower_left_arm"><material>Gazebo/Blue</material></gazebo>
+    <gazebo reference="lower_right_arm"><material>Gazebo/Blue</material></gazebo>
+    <gazebo reference="upper_left_arm"><material>Gazebo/Red</material></gazebo>
+    <gazebo reference="upper_right_arm"><material>Gazebo/Red</material></gazebo>
+    <gazebo reference="piston_actuator_link"><material>Gazebo/Black</material></gazebo>
+    <!-- Friction settings -->
     <gazebo reference="lift_link">
       <mu1>0.9</mu1><mu2>0.9</mu2>

Commit message: Fix scissor lift URDF structure and joint connections

File: src/mobile_lift_arm/urdf/scissor_lift.xacro (robot description, xacro)
@@ -3,155 +3,102 @@
   <!-- Include macros for inertia -->
   <xacro:include filename="$(find mobile_lift_arm)/urdf/scissor_lift_macros.xacro"/>
-  <!-- Parameters -->
-  <xacro:property name="base_length" value="1.0"/>
-  <xacro:property name="base_width" value="0.8"/>
-  <xacro:property name="base_height" value="0.1"/>
-  <xacro:property name="scissor_arm_length" value="0.8"/>
-  <xacro:property name="scissor_arm_width" value="0.05"/>
-  <xacro:property name="scissor_arm_height" value="0.03"/>
-  <xacro:property name="platform_length" value="0.9"/>
-  <xacro:property name="platform_width" value="0.7"/>
-  <xacro:property name="platform_height" value="0.05"/>
+  <!-- Parameters - Reduced size for mobile platform -->
+  <xacro:property name="base_length" value="0.6"/>
+  <xacro:property name="base_width" value="0.5"/>
+  <xacro:property name="base_height" value="0.05"/>
+  <xacro:property name="scissor_arm_length" value="0.4"/>
+  <xacro:property name="scissor_arm_width" value="0.03"/>
+  <xacro:property name="scissor_arm_height" value="0.02"/>
+  <xacro:property name="platform_length" value="0.5"/>
+  <xacro:property name="platform_width" value="0.4"/>
+  <xacro:property name="platform_height" value="0.03"/>
   <xacro:macro name="scissor_lift" params="parent">
-    <!-- Base Platform -->
-    <link name="lift_base">
+    <!-- Lift Link - Main platform that moves up/down -->
+    <link name="lift_link">
       <visual>
-        <geometry><box size="${base_length} ${base_width} ${base_height}"/></geometry>
-        <material name="grey"><color rgba="0.5 0.5 0.5 1"/></material>
+        <origin xyz="0 0 ${platform_height/2}" rpy="0 0 0"/>
+        <geometry><box size="${platform_length} ${platform_width} ${platform_height}"/></geometry>
+        <material name="green"><color rgba="0 0.8 0 1"/></material>
       </visual>
       <collision>
-        <geometry><box size="${base_length} ${base_width} ${base_height}"/></geometry>
-      </collision>
-      <xacro:box_inertia m="20" x="${base_length}" y="${base_width}" z="${base_height}"/>
-    </link>
-    <joint name="lift_base_joint" type="fixed">
-      <parent link="${parent}"/>
-      <child link="lift_base"/>
-      <origin xyz="0 0 0.1" rpy="0 0 0"/>
-    </joint>
-    <!-- === Left Side === -->
-    <link name="lower_left_arm">
-      <visual>
-        <geometry><box size="${scissor_arm_length} ${scissor_arm_width} ${scissor_arm_height}"/></geometry>
-        <material name="blue"><color rgba="0 0 1 1"/></material>
-      </visual>
-      <collision>
-        <geometry><box size="${scissor_arm_length} ${scissor_arm_width} ${scissor_arm_height}"/></geometry>
-      </collision>
-      <xacro:box_inertia m="2" x="${scissor_arm_length}" y="${scissor_arm_width}" z="${scissor_arm_height}"/>
-    </link>
-    <joint name="lower_left_joint" type="revolute">
-      <parent link="lift_base"/>
-      <child link="lower_left_arm"/>
-      <origin xyz="-${scissor_arm_length/2} -${base_width/4} ${base_height/2}"/>
-      <axis xyz="0 1 0"/>
-      <limit lower="0.0" upper="1.57" effort="500" velocity="1.0"/>
-      <dynamics damping="2.0" friction="0.1"/>
-    </joint>
-    <link name="upper_left_arm">
-      <visual>
-        <geometry><box size="${scissor_arm_length} ${scissor_arm_width} ${scissor_arm_height}"/></geometry>
-        <material name="red"><color rgba="1 0 0 1"/></material>
-      </visual>
-      <collision>
-        <geometry><box size="${scissor_arm_length} ${scissor_arm_width} ${scissor_arm_height}"/></geometry>
-      </collision>
-      <xacro:box_inertia m="2" x="${scissor_arm_length}" y="${scissor_arm_width}" z="${scissor_arm_height}"/>
-    </link>
-    <joint name="left_cross_joint" type="revolute">
-      <parent link="lower_left_arm"/>
-      <child link="upper_left_arm"/>
-      <origin xyz="0 0 0" rpy="0 0 0"/>
-      <axis xyz="0 1 0"/>
-      <limit lower="-3.14" upper="3.14" effort="500" velocity="1.0"/>
-      <dynamics damping="2.0" friction="0.1"/>
-    </joint>
-    <!-- === Right Side === -->
-    <link name="lower_right_arm">
-      <visual>
-        <geometry><box size="${scissor_arm_length} ${scissor_arm_width} ${scissor_arm_height}"/></geometry>
-        <material name="blue"/>
-      </visual>
-      <collision>
-        <geometry><box size="${scissor_arm_length} ${scissor_arm_width} ${scissor_arm_height}"/></geometry>
-      </collision>
-      <xacro:box_inertia m="2" x="${scissor_arm_length}" y="${scissor_arm_width}" z="${scissor_arm_height}"/>
-    </link>
-    <joint name="lower_right_joint" type="revolute">
-      <parent link="lift_base"/>
-      <child link="lower_right_arm"/>
-      <origin xyz="-${scissor_arm_length/2} ${base_width/4} ${base_height/2}"/>
-      <axis xyz="0 1 0"/>
-      <limit lower="0.0" upper="1.57" effort="500" velocity="1.0"/>
-      <dynamics damping="2.0" friction="0.1"/>
-    </joint>
-    <link name="upper_right_arm">
-      <visual>
-        <geometry><box size="${scissor_arm_length} ${scissor_arm_width} ${scissor_arm_height}"/></geometry>
-        <material name="red"/>
-      </visual>
-      <collision>
-        <geometry><box size="${scissor_arm_length} ${scissor_arm_width} ${scissor_arm_height}"/></geometry>
-      </collision>
-      <xacro:box_inertia m="2" x="${scissor_arm_length}" y="${scissor_arm_width}" z="${scissor_arm_height}"/>
-    </link>
-    <joint name="right_cross_joint" type="revolute">
-      <parent link="lower_right_arm"/>
-      <child link="upper_right_arm"/>
-      <origin xyz="0 0 0" rpy="0 0 0"/>
-      <axis xyz="0 1 0"/>
-      <limit lower="-3.14" upper="3.14" effort="500" velocity="1.0"/>
-      <dynamics damping="2.0" friction="0.1"/>
-    </joint>
-    <!-- === Lift Platform === -->
-    <link name="lift_link">
-      <visual>
-        <geometry><box size="${platform_length} ${platform_width} ${platform_height}"/></geometry>
-        <material name="green"><color rgba="0 1 0 1"/></material>
-      </visual>
-      <collision>
+        <origin xyz="0 0 ${platform_height/2}" rpy="0 0 0"/>
         <geometry><box size="${platform_length} ${platform_width} ${platform_height}"/></geometry>
       </collision>
       <xacro:box_inertia m="8" x="${platform_length}" y="${platform_width}" z="${platform_height}"/>
     </link>
-    <joint name="platform_left_joint" type="revolute">
-      <parent link="upper_left_arm"/>
+    <!-- Main lift joint - Simple prismatic for now -->
+    <joint name="lift_joint" type="prismatic">
+      <parent link="${parent}"/>
       <child link="lift_link"/>
-      <origin xyz="${scissor_arm_length/2} 0 ${platform_height/2}"/>
+      <origin xyz="0 0 0.15" rpy="0 0 0"/>
+      <axis xyz="0 0 1"/>
+      <limit lower="0.0" upper="1.2" effort="2000" velocity="0.5"/>
+      <dynamics damping="10.0" friction="0.2"/>
+    </joint>
+    <!-- Scissor mechanism base -->
+    <link name="scissor_base">
+      <visual>
+        <origin xyz="0 0 ${base_height/2}" rpy="0 0 0"/>
+        <geometry><box size="${base_length} ${base_width} ${base_height}"/></geometry>
+        <material name="grey"><color rgba="0.6 0.6 0.6 1"/></material>
+      </visual>
+      <collision>
+        <origin xyz="0 0 ${base_height/2}" rpy="0 0 0"/>
+        <geometry><box size="${base_length} ${base_width} ${base_height}"/></geometry>
+      </collision>
+      <xacro:box_inertia m="5" x="${base_length}" y="${base_width}" z="${base_height}"/>
+    </link>
+    <joint name="scissor_base_joint" type="fixed">
+      <parent link="${parent}"/>
+      <child link="scissor_base"/>
+      <origin xyz="0 0 0.05" rpy="0 0 0"/>
+    </joint>
+    <!-- Left scissor arm -->
+    <link name="left_scissor_arm">
+      <visual>
+        <origin xyz="0 0 0" rpy="0 0 0"/>
+        <geometry><box size="${scissor_arm_length} ${scissor_arm_width} ${scissor_arm_height}"/></geometry>
+        <material name="blue"><color rgba="0.2 0.2 0.8 1"/></material>
+      </visual>
+      <collision>
+        <origin xyz="0 0 0" rpy="0 0 0"/>
+        <geometry><box size="${scissor_arm_length} ${scissor_arm_width} ${scissor_arm_height}"/></geometry>
+      </collision>
+      <xacro:box_inertia m="1" x="${scissor_arm_length}" y="${scissor_arm_width}" z="${scissor_arm_height}"/>
+    </link>
+    <joint name="left_scissor_joint" type="revolute">
+      <parent link="scissor_base"/>
+      <child link="left_scissor_arm"/>
+      <origin xyz="-${base_length/4} -${base_width/4} ${base_height}" rpy="0 0 0"/>
       <axis xyz="0 1 0"/>
-      <limit lower="-3.14" upper="3.14" effort="500" velocity="1.0"/>
+      <limit lower="0.0" upper="1.57" effort="500" velocity="2.0"/>
       <dynamics damping="2.0" friction="0.1"/>
     </joint>
-    <joint name="platform_right_joint" type="fixed">
-      <parent link="lift_link"/>
-      <child link="upper_right_arm"/>
-      <origin xyz="0 -${base_width/2} 0" rpy="0 0 0"/>
-    </joint>
-    <!-- === Hydraulic Actuator === -->
-    <link name="piston_actuator_link">
+    <!-- Right scissor arm -->
+    <link name="right_scissor_arm">
       <visual>
-        <geometry><cylinder length="0.1" radius="0.02"/></geometry>
-        <material name="black"><color rgba="0.2 0.2 0.2 1"/></material>
+        <origin xyz="0 0 0" rpy="0 0 0"/>
+        <geometry><box size="${scissor_arm_length} ${scissor_arm_width} ${scissor_arm_height}"/></geometry>
+        <material name="blue"><color rgba="0.2 0.2 0.8 1"/></material>
       </visual>
       <collision>
-        <geometry><cylinder length="0.1" radius="0.02"/></geometry>
+        <origin xyz="0 0 0" rpy="0 0 0"/>
+        <geometry><box size="${scissor_arm_length} ${scissor_arm_width} ${scissor_arm_height}"/></geometry>
       </collision>
-      <xacro:cylinder_inertia m="1" r="0.02" l="0.1"/>
+      <xacro:box_inertia m="1" x="${scissor_arm_length}" y="${scissor_arm_width}" z="${scissor_arm_height}"/>
     </link>
-    <joint name="lift_joint" type="prismatic">
-      <parent link="lift_base"/>
-      <child link="piston_actuator_link"/>
-      <origin xyz="0 0 ${base_height/2}" rpy="0 0 0"/>
-      <axis xyz="1 0 0"/>
-      <limit lower="-0.3" upper="0.3" effort="2000" velocity="0.2"/>
-      <dynamics damping="10.0" friction="0.2"/>
+    <joint name="right_scissor_joint" type="revolute">
+      <parent link="scissor_base"/>
+      <child link="right_scissor_arm"/>
+      <origin xyz="-${base_length/4} ${base_width/4} ${base_height}" rpy="0 0 0"/>
+      <axis xyz="0 1 0"/>
+      <limit lower="0.0" upper="1.57" effort="500" velocity="2.0"/>
+      <dynamics damping="2.0" friction="0.1"/>
     </joint>
-    <joint name="actuator_to_left_arm" type="revolute">
-        <parent link="piston_actuator_link"/>
-        <child link="lower_left_arm"/>
-        <origin xyz="0 0 0" rpy="0 0 0"/>
-        <axis xyz="0 1 0"/>
-        <limit lower="-3.14" upper="3.14" effort="500" velocity="1.0"/>
-        <dynamics damping="2.0" friction="0.1"/>
+    <!-- Connect scissor arms to platform (visual connection) -->
+    <joint name="left_arm_to_platform" type="fixed">
+      <parent link="left_scissor_arm"/>
+      <child link="lift_link"/>
+      <origin xyz="${scissor_arm_length/2} ${base_width/2} 0.1" rpy="0 0 0"/>
     </joint>
     <!-- Top link for arm attachment -->
@@ -160,14 +107,11 @@
       <parent link="lift_link"/>
       <child link="lift_top_link"/>
-      <origin xyz="0 0 ${platform_height/2}" rpy="0 0 0"/>
+      <origin xyz="0 0 ${platform_height}" rpy="0 0 0"/>
     </joint>
     <!-- Gazebo materials -->
-    <gazebo reference="lift_base"><material>Gazebo/Grey</material></gazebo>
     <gazebo reference="lift_link"><material>Gazebo/Green</material></gazebo>
-    <gazebo reference="lower_left_arm"><material>Gazebo/Blue</material></gazebo>
-    <gazebo reference="lower_right_arm"><material>Gazebo/Blue</material></gazebo>
-    <gazebo reference="upper_left_arm"><material>Gazebo/Red</material></gazebo>
-    <gazebo reference="upper_right_arm"><material>Gazebo/Red</material></gazebo>
-    <gazebo reference="piston_actuator_link"><material>Gazebo/Black</material></gazebo>
+    <gazebo reference="scissor_base"><material>Gazebo/Grey</material></gazebo>
+    <gazebo reference="left_scissor_arm"><material>Gazebo/Blue</material></gazebo>
+    <gazebo reference="right_scissor_arm"><material>Gazebo/Blue</material></gazebo>
     <!-- Friction settings -->
     <gazebo reference="lift_link">
