Commit message: Fix kinematic structure: remove kinematic loops, simplify scissor mechanism

File: src/mobile_lift_arm/urdf/scissor_lift.xacro (robot description, xacro)
@@ -3,5 +3,7 @@
   <!-- Include macros for inertia -->
   <xacro:include filename="$(find mobile_lift_arm)/urdf/scissor_lift_macros.xacro"/>
-  <!-- Parameters - Reduced size for mobile platform -->
+  <!-- Parameters - Optimized for mobile platform -->
+  <xacro:property name="LIFT_MIN" value="0.0"/>
+  <xacro:property name="LIFT_MAX" value="1.2"/>
   <xacro:property name="base_length" value="0.6"/>
   <xacro:property name="base_width" value="0.5"/>
@@ -14,26 +16,4 @@
   <xacro:property name="platform_height" value="0.03"/>
   <xacro:macro name="scissor_lift" params="parent">
-    <!-- Lift Link - Main platform that moves up/down -->
-    <link name="lift_link">
-      <visual>
-        <origin xyz="0 0 ${platform_height/2}" rpy="0 0 0"/>
-        <geometry><box size="${platform_length} ${platform_width} ${platform_height}"/></geometry>
-        <material name="green"><color rgba="0 0.8 0 1"/></material>
-      </visual>
-      <collision>
-        <origin xyz="0 0 ${platform_height/2}" rpy="0 0 0"/>
-        <geometry><box size="${platform_length} ${platform_width} ${platform_height}"/></geometry>
-      </collision>
-      <xacro:box_inertia m="8" x="${platform_length}" y="${platform_width}" z="${platform_height}"/>
-    </link>
-    <!-- Main lift joint - Simple prismatic for now -->
-    <joint name="lift_joint" type="prismatic">
-      <parent link="${parent}"/>
-      <child link="lift_link"/>
-      <origin xyz="0 0 0.15" rpy="0 0 0"/>
-      <axis xyz="0 0 1"/>
-      <limit lower="0.0" upper="1.2" effort="2000" velocity="0.5"/>
-      <dynamics damping="10.0" friction="0.2"/>
-    </joint>
     <!-- Scissor mechanism base -->
     <link name="scissor_base">
@@ -54,53 +34,81 @@
       <origin xyz="0 0 0.05" rpy="0 0 0"/>
     </joint>
-    <!-- Left scissor arm -->
+    <!-- Main Lift Platform - This moves up and down -->
+    <link name="lift_link">
+      <visual>
+        <origin xyz="0 0 ${platform_height/2}" rpy="0 0 0"/>
+        <geometry><box size="${platform_length} ${platform_width} ${platform_height}"/></geometry>
+        <material name="green"><color rgba="0 0.8 0 1"/></material>
+      </visual>
+      <collision>
+        <origin xyz="0 0 ${platform_height/2}" rpy="0 0 0"/>
+        <geometry><box size="${platform_length} ${platform_width} ${platform_height}"/></geometry>
+      </collision>
+      <xacro:box_inertia m="8" x="${platform_length}" y="${platform_width}" z="${platform_height}"/>
+    </link>
+    <!-- Main lift joint - This is controlled by the position controller -->
+    <joint name="lift_joint" type="prismatic">
+      <parent link="scissor_base"/>
+      <child link="lift_link"/>
+      <origin xyz="0 0 ${base_height + 0.1}" rpy="0 0 0"/>
+      <axis xyz="0 0 1"/>
+      <limit lower="${LIFT_MIN}" upper="${LIFT_MAX}" effort="2000" velocity="0.5"/>
+      <dynamics damping="10.0" friction="0.2"/>
+    </joint>
+    <!-- Visual Scissor Arms (fixed for appearance) -->
     <link name="left_scissor_arm">
       <visual>
-        <origin xyz="0 0 0" rpy="0 0 0"/>
+        <origin xyz="0 0 0" rpy="0 0 0.785"/>
         <geometry><box size="${scissor_arm_length} ${scissor_arm_width} ${scissor_arm_height}"/></geometry>
         <material name="blue"><color rgba="0.2 0.2 0.8 1"/></material>
       </visual>
       <collision>
-        <origin xyz="0 0 0" rpy="0 0 0"/>
+        <origin xyz="0 0 0" rpy="0 0 0.785"/>
         <geometry><box size="${scissor_arm_length} ${scissor_arm_width} ${scissor_arm_height}"/></geometry>
       </collision>
       <xacro:box_inertia m="1" x="${scissor_arm_length}" y="${scissor_arm_width}" z="${scissor_arm_height}"/>
     </link>
-    <joint name="left_scissor_joint" type="revolute">
+    <joint name="left_scissor_joint" type="fixed">
       <parent link="scissor_base"/>
       <child link="left_scissor_arm"/>
-      <origin xyz="-${base_length/4} -${base_width/4} ${base_height}" rpy="0 0 0"/>
-      <axis xyz="0 1 0"/>
-      <limit lower="0.0" upper="1.57" effort="500" velocity="2.0"/>
-      <dynamics damping="2.0" friction="0.1"/>
+      <origin xyz="-${base_length/4} -${base_width/4} ${base_height + 0.3}" rpy="0 0 0"/>
     </joint>
     <!-- Right scissor arm -->
     <link name="right_scissor_arm">
       <visual>
-        <origin xyz="0 0 0" rpy="0 0 0"/>
+        <origin xyz="0 0 0" rpy="0 0 -0.785"/>
         <geometry><box size="${scissor_arm_length} ${scissor_arm_width} ${scissor_arm_height}"/></geometry>
-        <material name="blue"><color rgba="0.2 0.2 0.8 1"/></material>
+        <material name="red"><color rgba="0.8 0.2 0.2 1"/></material>
       </visual>
       <collision>
-        <origin xyz="0 0 0" rpy="0 0 0"/>
+        <origin xyz="0 0 0" rpy="0 0 -0.785"/>
         <geometry><box size="${scissor_arm_length} ${scissor_arm_width} ${scissor_arm_height}"/></geometry>
       </collision>
       <xacro:box_inertia m="1" x="${scissor_arm_length}" y="${scissor_arm_width}" z="${scissor_arm_height}"/>
     </link>
-    <joint name="right_scissor_joint" type="revolute">
+    <joint name="right_scissor_joint" type="fixed">
       <parent link="scissor_base"/>
       <child link="right_scissor_arm"/>
-      <origin xyz="-${base_length/4} ${base_width/4} ${base_height}" rpy="0 0 0"/>
-      <axis xyz="0 1 0"/>
-      <limit lower="0.0" upper="1.57" effort="500" velocity="2.0"/>
-      <dynamics damping="2.0" friction="0.1"/>
+      <origin xyz="-${base_length/4} ${base_width/4} ${base_height + 0.3}" rpy="0 0 0"/>
     </joint>
-    <!-- Connect scissor arms to platform (visual connection) -->
-    <joint name="left_arm_to_platform" type="fixed">
-      <parent link="left_scissor_arm"/>
-      <child link="lift_link"/>
-      <origin xyz="${scissor_arm_length/2} ${base_width/2} 0.1" rpy="0 0 0"/>
+    <!-- Hydraulic cylinder visual -->
+    <link name="hydraulic_cylinder">
+      <visual>
+        <origin xyz="0 0 0" rpy="0 0 0"/>
+        <geometry><cylinder length="0.3" radius="0.025"/></geometry>
+        <material name="black"><color rgba="0.2 0.2 0.2 1"/></material>
+      </visual>
+      <collision>
+        <origin xyz="0 0 0" rpy="0 0 0"/>
+        <geometry><cylinder length="0.3" radius="0.025"/></geometry>
+      </collision>
+      <xacro:cylinder_inertia m="2" r="0.025" l="0.3"/>
+    </link>
+    <joint name="cylinder_joint" type="fixed">
+      <parent link="scissor_base"/>
+      <child link="hydraulic_cylinder"/>
+      <origin xyz="0.2 0 0.25" rpy="0 0 0"/>
     </joint>
-    <!-- Top link for arm attachment -->
+    <!-- Top attachment point for robot arm -->
     <link name="lift_top_link"/>
     <joint name="lift_top_fixed" type="fixed">
@@ -113,5 +121,6 @@
     <gazebo reference="scissor_base"><material>Gazebo/Grey</material></gazebo>
     <gazebo reference="left_scissor_arm"><material>Gazebo/Blue</material></gazebo>
-    <gazebo reference="right_scissor_arm"><material>Gazebo/Blue</material></gazebo>
+    <gazebo reference="right_scissor_arm"><material>Gazebo/Red</material></gazebo>
+    <gazebo reference="hydraulic_cylinder"><material>Gazebo/Black</material></gazebo>
     <!-- Friction settings -->
     <gazebo reference="lift_link">

Commit message: Fix scissor lift positioning: place correctly between base and arm

File: src/mobile_lift_arm/urdf/scissor_lift.xacro (robot description, xacro)
@@ -6,20 +6,20 @@
   <xacro:property name="LIFT_MIN" value="0.0"/>
   <xacro:property name="LIFT_MAX" value="1.2"/>
-  <xacro:property name="base_length" value="0.6"/>
-  <xacro:property name="base_width" value="0.5"/>
-  <xacro:property name="base_height" value="0.05"/>
-  <xacro:property name="scissor_arm_length" value="0.4"/>
-  <xacro:property name="scissor_arm_width" value="0.03"/>
-  <xacro:property name="scissor_arm_height" value="0.02"/>
-  <xacro:property name="platform_length" value="0.5"/>
-  <xacro:property name="platform_width" value="0.4"/>
-  <xacro:property name="platform_height" value="0.03"/>
+  <xacro:property name="base_length" value="0.8"/>
+  <xacro:property name="base_width" value="0.6"/>
+  <xacro:property name="base_height" value="0.08"/>
+  <xacro:property name="scissor_arm_length" value="0.5"/>
+  <xacro:property name="scissor_arm_width" value="0.04"/>
+  <xacro:property name="scissor_arm_height" value="0.03"/>
+  <xacro:property name="platform_length" value="0.7"/>
+  <xacro:property name="platform_width" value="0.5"/>
+  <xacro:property name="platform_height" value="0.05"/>
   <xacro:macro name="scissor_lift" params="parent">
-    <!-- Scissor mechanism base -->
+    <!-- Scissor mechanism base platform -->
     <link name="scissor_base">
       <visual>
         <origin xyz="0 0 ${base_height/2}" rpy="0 0 0"/>
         <geometry><box size="${base_length} ${base_width} ${base_height}"/></geometry>
-        <material name="grey"><color rgba="0.6 0.6 0.6 1"/></material>
+        <material name="dark_grey"><color rgba="0.3 0.3 0.3 1"/></material>
       </visual>
       <collision>
@@ -29,8 +29,80 @@
       <xacro:box_inertia m="5" x="${base_length}" y="${base_width}" z="${base_height}"/>
     </link>
+    <!-- Mount scissor base DIRECTLY on top of the vehicle base -->
     <joint name="scissor_base_joint" type="fixed">
       <parent link="${parent}"/>
       <child link="scissor_base"/>
-      <origin xyz="0 0 0.05" rpy="0 0 0"/>
+      <origin xyz="0 0 0.18" rpy="0 0 0"/>
+    </joint>
+    <!-- Visual Scissor Arms positioned correctly -->
+    <link name="left_scissor_arm">
+      <visual>
+        <origin xyz="0 0 0" rpy="0 0 0.5"/>
+        <geometry><box size="${scissor_arm_length} ${scissor_arm_width} ${scissor_arm_height}"/></geometry>
+        <material name="blue"><color rgba="0.2 0.4 0.8 1"/></material>
+      </visual>
+      <collision>
+        <origin xyz="0 0 0" rpy="0 0 0.5"/>
+        <geometry><box size="${scissor_arm_length} ${scissor_arm_width} ${scissor_arm_height}"/></geometry>
+      </collision>
+      <xacro:box_inertia m="1" x="${scissor_arm_length}" y="${scissor_arm_width}" z="${scissor_arm_height}"/>
+    </link>
+    <joint name="left_scissor_joint" type="fixed">
+      <parent link="scissor_base"/>
+      <child link="left_scissor_arm"/>
+      <origin xyz="-0.15 -0.1 ${base_height + 0.15}" rpy="0 0 0"/>
+    </joint>
+    <!-- Right scissor arm -->
+    <link name="right_scissor_arm">
+      <visual>
+        <origin xyz="0 0 0" rpy="0 0 -0.5"/>
+        <geometry><box size="${scissor_arm_length} ${scissor_arm_width} ${scissor_arm_height}"/></geometry>
+        <material name="red"><color rgba="0.8 0.2 0.2 1"/></material>
+      </visual>
+      <collision>
+        <origin xyz="0 0 0" rpy="0 0 -0.5"/>
+        <geometry><box size="${scissor_arm_length} ${scissor_arm_width} ${scissor_arm_height}"/></geometry>
+      </collision>
+      <xacro:box_inertia m="1" x="${scissor_arm_length}" y="${scissor_arm_width}" z="${scissor_arm_height}"/>
+    </link>
+    <joint name="right_scissor_joint" type="fixed">
+      <parent link="scissor_base"/>
+      <child link="right_scissor_arm"/>
+      <origin xyz="-0.15 0.1 ${base_height + 0.15}" rpy="0 0 0"/>
+    </joint>
+    <!-- Upper scissor arms -->
+    <link name="upper_left_scissor_arm">
+      <visual>
+        <origin xyz="0 0 0" rpy="0 0 -0.5"/>
+        <geometry><box size="${scissor_arm_length} ${scissor_arm_width} ${scissor_arm_height}"/></geometry>
+        <material name="blue"/>
+      </visual>
+      <collision>
+        <origin xyz="0 0 0" rpy="0 0 -0.5"/>
+        <geometry><box size="${scissor_arm_length} ${scissor_arm_width} ${scissor_arm_height}"/></geometry>
+      </collision>
+      <xacro:box_inertia m="1" x="${scissor_arm_length}" y="${scissor_arm_width}" z="${scissor_arm_height}"/>
+    </link>
+    <joint name="upper_left_scissor_joint" type="fixed">
+      <parent link="scissor_base"/>
+      <child link="upper_left_scissor_arm"/>
+      <origin xyz="0.15 -0.1 ${base_height + 0.15}" rpy="0 0 0"/>
+    </joint>
+    <link name="upper_right_scissor_arm">
+      <visual>
+        <origin xyz="0 0 0" rpy="0 0 0.5"/>
+        <geometry><box size="${scissor_arm_length} ${scissor_arm_width} ${scissor_arm_height}"/></geometry>
+        <material name="red"/>
+      </visual>
+      <collision>
+        <origin xyz="0 0 0" rpy="0 0 0.5"/>
+        <geometry><box size="${scissor_arm_length} ${scissor_arm_width} ${scissor_arm_height}"/></geometry>
+      </collision>
+      <xacro:box_inertia m="1" x="${scissor_arm_length}" y="${scissor_arm_width}" z="${scissor_arm_height}"/>
+    </link>
+    <joint name="upper_right_scissor_joint" type="fixed">
+      <parent link="scissor_base"/>
+      <child link="upper_right_scissor_arm"/>
+      <origin xyz="0.15 0.1 ${base_height + 0.15}" rpy="0 0 0"/>
     </joint>
     <!-- Main Lift Platform - This moves up and down -->
@@ -51,62 +123,43 @@
       <parent link="scissor_base"/>
       <child link="lift_link"/>
-      <origin xyz="0 0 ${base_height + 0.1}" rpy="0 0 0"/>
+      <origin xyz="0 0 ${base_height + 0.05}" rpy="0 0 0"/>
       <axis xyz="0 0 1"/>
       <limit lower="${LIFT_MIN}" upper="${LIFT_MAX}" effort="2000" velocity="0.5"/>
       <dynamics damping="10.0" friction="0.2"/>
     </joint>
-    <!-- Visual Scissor Arms (fixed for appearance) -->
-    <link name="left_scissor_arm">
-      <visual>
-        <origin xyz="0 0 0" rpy="0 0 0.785"/>
-        <geometry><box size="${scissor_arm_length} ${scissor_arm_width} ${scissor_arm_height}"/></geometry>
-        <material name="blue"><color rgba="0.2 0.2 0.8 1"/></material>
-      </visual>
-      <collision>
-        <origin xyz="0 0 0" rpy="0 0 0.785"/>
-        <geometry><box size="${scissor_arm_length} ${scissor_arm_width} ${scissor_arm_height}"/></geometry>
-      </collision>
-      <xacro:box_inertia m="1" x="${scissor_arm_length}" y="${scissor_arm_width}" z="${scissor_arm_height}"/>
-    </link>
-    <joint name="left_scissor_joint" type="fixed">
-      <parent link="scissor_base"/>
-      <child link="left_scissor_arm"/>
-      <origin xyz="-${base_length/4} -${base_width/4} ${base_height + 0.3}" rpy="0 0 0"/>
-    </joint>
-    <!-- Right scissor arm -->
-    <link name="right_scissor_arm">
-      <visual>
-        <origin xyz="0 0 0" rpy="0 0 -0.785"/>
-        <geometry><box size="${scissor_arm_length} ${scissor_arm_width} ${scissor_arm_height}"/></geometry>
-        <material name="red"><color rgba="0.8 0.2 0.2 1"/></material>
-      </visual>
-      <collision>
-        <origin xyz="0 0 0" rpy="0 0 -0.785"/>
-        <geometry><box size="${scissor_arm_length} ${scissor_arm_width} ${scissor_arm_height}"/></geometry>
-      </collision>
-      <xacro:box_inertia m="1" x="${scissor_arm_length}" y="${scissor_arm_width}" z="${scissor_arm_height}"/>
-    </link>
-    <joint name="right_scissor_joint" type="fixed">
-      <parent link="scissor_base"/>
-      <child link="right_scissor_arm"/>
-      <origin xyz="-${base_length/4} ${base_width/4} ${base_height + 0.3}" rpy="0 0 0"/>
-    </joint>
-    <!-- Hydraulic cylinder visual -->
-    <link name="hydraulic_cylinder">
+    <!-- Hydraulic cylinders for visual effect -->
+    <link name="hydraulic_cylinder_1">
       <visual>
         <origin xyz="0 0 0" rpy="0 0 0"/>
-        <geometry><cylinder length="0.3" radius="0.025"/></geometry>
+        <geometry><cylinder length="0.4" radius="0.02"/></geometry>
         <material name="black"><color rgba="0.2 0.2 0.2 1"/></material>
       </visual>
       <collision>
         <origin xyz="0 0 0" rpy="0 0 0"/>
-        <geometry><cylinder length="0.3" radius="0.025"/></geometry>
+        <geometry><cylinder length="0.4" radius="0.02"/></geometry>
       </collision>
-      <xacro:cylinder_inertia m="2" r="0.025" l="0.3"/>
+      <xacro:cylinder_inertia m="1" r="0.02" l="0.4"/>
     </link>
-    <joint name="cylinder_joint" type="fixed">
+    <joint name="cylinder_1_joint" type="fixed">
       <parent link="scissor_base"/>
-      <child link="hydraulic_cylinder"/>
-      <origin xyz="0.2 0 0.25" rpy="0 0 0"/>
+      <child link="hydraulic_cylinder_1"/>
+      <origin xyz="0.25 -0.15 0.3" rpy="0 0 0"/>
+    </joint>
+    <link name="hydraulic_cylinder_2">
+      <visual>
+        <origin xyz="0 0 0" rpy="0 0 0"/>
+        <geometry><cylinder length="0.4" radius="0.02"/></geometry>
+        <material name="black"/>
+      </visual>
+      <collision>
+        <origin xyz="0 0 0" rpy="0 0 0"/>
+        <geometry><cylinder length="0.4" radius="0.02"/></geometry>
+      </collision>
+      <xacro:cylinder_inertia m="1" r="0.02" l="0.4"/>
+    </link>
+    <joint name="cylinder_2_joint" type="fixed">
+      <parent link="scissor_base"/>
+      <child link="hydraulic_cylinder_2"/>
+      <origin xyz="0.25 0.15 0.3" rpy="0 0 0"/>
     </joint>
     <!-- Top attachment point for robot arm -->
@@ -122,5 +175,8 @@
     <gazebo reference="left_scissor_arm"><material>Gazebo/Blue</material></gazebo>
     <gazebo reference="right_scissor_arm"><material>Gazebo/Red</material></gazebo>
-    <gazebo reference="hydraulic_cylinder"><material>Gazebo/Black</material></gazebo>
+    <gazebo reference="upper_left_scissor_arm"><material>Gazebo/Blue</material></gazebo>
+    <gazebo reference="upper_right_scissor_arm"><material>Gazebo/Red</material></gazebo>
+    <gazebo reference="hydraulic_cylinder_1"><material>Gazebo/Black</material></gazebo>
+    <gazebo reference="hydraulic_cylinder_2"><material>Gazebo/Black</material></gazebo>
     <!-- Friction settings -->
     <gazebo reference="lift_link">
